File: RTM/2026.1/KiCad/TS_READY_TO_MOVE (1).kicad_sch (KiCad schematic)
At the start: 43 parts, among them J1 V_BIAS TEST, J2 Conn_01x02, J3 12V TEST, J4 V_IN TEST, J5 Conn_01x02, J7 Conn_01x02, Q2 NMOS, Q4 NMOS, Q5 NMOS, U1 MMSZ5245BT1G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

Commit message: 2026.1 fixed vbias, removed nmos after r9, r10/r8 increase
Parts:
- R10, R8: Note (none) -> Change to 24k, 0.125W, 0805
- renumbered RX to R2
Changed lines of the file:
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@@
 		(on_board yes)
 		(dnp no)
-		(property "Reference" "RX"
+		(property "Reference" "R2"
 			(at 221.742 134.366 0)
 			(effects
@@
 			(project "TS_READY_TO_MOVE (1)"
 				(path "/ec2b8551-75c2-4864-b31d-b681332831c2"
-					(reference "RX")
+					(reference "R2")
 					(unit 1)
 				)
@@
 			)
 		)
+		(property "Note" "Change to 24k, 0.125W, 0805"
+			(at 158.75 49.53 0)
+			(effects
+				(font
+					(size 1.27 1.27)
+				)
+				(hide yes)
+			)
+		)
 		(pin "1"
 		)
@@
 			(at 167.64 49.53 0)
 			(effects
+				(font
+					(size 1.27 1.27)
+				)
+				(hide yes)
+			)
+		)
+		(property "Note" "Change to 24k, 0.125W, 0805"
+			(at 167.64 49.53 0)
+			(effects
