File: RTM/2026.1/KiCad/TS_READY_TO_MOVE (1).kicad_pcb (KiCad board)
At the start: 2 copper layers, 71 x 54.8 mm, 43 parts, among them J2 Conn_01x02, J5 Conn_01x02, J7 Conn_01x02, Q2 NMOS, Q3 NMOS, Q4 NMOS, Q5 NMOS, U1 MMSZ5245BT1G, U2 4N35, U3 LM555xN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

Commit message: 2026.1 fixed vbias, removed nmos after r9, r10/r8 increase
Parts:
- removed Q3: NMOS, Package_TO_SOT_THT:TO-220-3_Vertical
- added R2: 11k, Resistor_SMD:R_0805_2012Metric, F.Cu at (53.3, 67.0)
- moved R17 0.39 mm to (55.9, 67.7)
- renumbered V_BIAS to J1, 12V to J3, V_IN to J4
Connections:
- J4 pad 1: 12V_UNISO -> (no net)
- R9 pad 2: Net-(Q3-D) -> (no net)
- RV1 pad 3: 12V_UNISO -> V_BIAS
- U4 pad 2: 12V_UNISO -> V_BIAS
Routing:
- net V_BIAS: track 0.00 -> 60.1 mm
- net 12V_UNISO: track 100.8 -> 86.0 mm
- net Net-(Q3-D): track 10.9 -> 0.00 mm
- net Net-(DEBUG_1-K): track 57.1 -> 53.3 mm, vias 0 -> 1
- net Net-(Q2-D): track 16.2 -> 17.7 mm
- net Net-(R9-Pad2): track 28.5 -> 29.0 mm, vias 0 -> 1
- net (no net): vias 0 -> 1

Commit message: Updated RTM silkscreen
Parts:
- renumbered DEBUG_1 to DEBUG_LED_1, DEBUG_2 to DEBUG_LED_2, DEBUG_3 to DEBUG_LED_3
Other:
- board text added: "+12V_UNISO"
- board text added: "ANODE"
- board text added: "CATHODE"
- board text added: "GND"
- board text added: "HV+"
- board text added: "HV-"
- board text added: "VCC"
- board text added: "V_BIAS"
- board text added: "V_IN"
Changed lines of the file:
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@@
 		(descr "LED, diameter 5.0mm, 2 pins, http://cdn-reichelt.de/documents/datenblatt/A500/LL-504BC2E-009.pdf")
 		(tags "LED diameter 5.0mm 2 pins")
-		(property "Reference" "DEBUG_1"
-			(at 0.971847 -4.18 180)
+		(property "Reference" "DEBUG_LED_1"
+			(at -0.528153 4.32 180)
 			(layer "F.SilkS")
 			(effects
@@
 		(descr "LED, diameter 5.0mm, 2 pins, http://cdn-reichelt.de/documents/datenblatt/A500/LL-504BC2E-009.pdf")
 		(tags "LED diameter 5.0mm 2 pins")
-		(property "Reference" "DEBUG_3"
+		(property "Reference" "DEBUG_LED_3"
 			(at 1.343153 4.18 0)
 			(layer "F.SilkS")
@@
 		(tags "resistor")
 		(property "Reference" "R1"
-			(at 0 -1.65 0)
+			(at 0 1.5925 0)
 			(layer "F.SilkS")
 			(effects
@@
 		(descr "LED, diameter 5.0mm, 2 pins, http://cdn-reichelt.de/documents/datenblatt/A500/LL-504BC2E-009.pdf")
 		(tags "LED diameter 5.0mm 2 pins")
-		(property "Reference" "DEBUG_2"
+		(property "Reference" "DEBUG_LED_2"
 			(at 1.268153 4.18 0)
 			(layer "F.SilkS")
@@
 		(tags "connector Molex Mini-Fit_Jr side entryplastic_peg")
 		(property "Reference" "J7"
-			(at 0 -3.45 0)
+			(at 0 -5.21 0)
 			(layer "F.SilkS")
 			(effects
@@
 		(layer "Edge.Cuts")
 	)
+	(gr_text "ANODE"
+		(at 78 29 90)
+		(layer "F.SilkS")
+		(effects
+			(font
+				(size 1 1)
+				(thickness 0.1)
+			)
+			(justify left bottom)
+		)
+	)
+	(gr_text "V_IN"
+		(at 62 43 90)
+		(layer "F.SilkS")
+		(effects
+			(font
+				(size 1 0.75)
+				(thickness 0.1)
+			)
+			(justify left bottom)
+		)
+	)
+	(gr_text "HV+"
+		(at 32.5 28.5 90)
+		(layer "F.SilkS")
+		(effects
+			(font
+				(size 1 1)
+				(thickness 0.1)
+			)
+			(justify left bottom)
+		)
+	)
 	(gr_text "NON-ISOLATED"
 		(at 61.5 22.25 270)
@@
 	)
 	(gr_text "LV CONNECTOR"
-		(at 22.75 56.5 0)
+		(at 22.75 58 0)
+		(layer "F.SilkS")
+		(effects
+			(font
+				(size 1 1)
+				(thickness 0.1)
+			)
+			(justify left bottom)
+		)
+	)
+	(gr_text "CATHODE"
+		(at 81.5 36 90)
+		(layer "F.SilkS")
+		(effects
+			(font
+				(size 1 1)
+				(thickness 0.1)
+			)
+			(justify left bottom)
+		)
+	)
+	(gr_text "VCC"
+		(at 77 41 90)
+		(layer "F.SilkS")
+		(effects
+			(font
+				(size 1 1)
+				(thickness 0.1)
+			)
+			(justify left bottom)
+		)
+	)
+	(gr_text "GND"
+		(at 27 56.5 0)
+		(layer "F.SilkS")
+		(effects
+			(font
+				(size 1 1)
+				(thickness 0.1)
+			)
+			(justify left bottom)
+		)
+	)
+	(gr_text "+12V_UNISO"
+		(at 23.5 42.5 0)
 		(layer "F.SilkS")
 		(effects
@@
 		)
 	)
+	(gr_text "V_BIAS"
+		(at 62 46.5 90)
+		(layer "F.SilkS")
+		(effects
+			(font
+				(size 1 0.5)
+				(thickness 0.1)
+			)
+			(justify left bottom)
+		)
+	)
 	(gr_text "ISOLATED"
 		(at 66 33 90)
@@
 		(layer "F.SilkS")
 		(effects
+			(font
+				(size 1 1)
+				(thickness 0.1)
+			)
+			(justify left bottom)
+		)
+	)
+	(gr_text "HV-"
+		(at 29.5 33.5 90)
+		(layer "F.SilkS")
+		(effects
+			(font
+				(size 1 1)
+				(thickness 0.1)
+			)
+			(justify left bottom)
+		)
+	)
+	(gr_text "GND"
+		(at 65 41 90)
+		(layer "F.SilkS")
+		(effects
