File: TSSI/2026.2/KiCad/TSSI2026.2.kicad_pcb (KiCad board)
At the start: 2 copper layers, 66 x 35 mm, 31 parts, among them J2 Conn_01x02, J3 Conn_02x02, Q1 IRLZ34N, T555 Test555, U1 LM555xN, U2 IRLZ34N, U3 IRLZ34N, U4 4001, U5 4069

Commit message: Add silkscreen
Other:
- board text added: "Green"
- board text added: "Red"
Changed lines of the file:
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@@
+		)
+	)
+	(gr_text "Green"
+		(at 86 47 0)
+		(layer "F.SilkS")
+		(effects
+			(font
+				(size 1 1)
+				(thickness 0.25)
+				(bold yes)
+			)
+			(justify left bottom)
+		)
+	)
+	(gr_text "Red"
+		(at 92 47 0)
+		(layer "F.SilkS")
+		(effects
+			(font
+				(size 1 1)
+				(thickness 0.25)
+				(bold yes)
+			)
+			(justify left bottom)
 		)
 	)
