File: RTM/2026.2/RTM.kicad_pcb (KiCad board)
At the start: 2 copper layers, 71 x 54.8 mm, 45 parts, among them J1 V_BIAS TEST, J2 Conn_01x02, J3 12V TEST, J4 V_IN TEST, J5 Conn_01x02, J7 Conn_01x02, Q2 NMOS, Q4 NMOS, Q5 NMOS, U1 MMSZ5245BT1G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

Commit message: Add files via upload
Parts:
- R1, R11, R12, R16, R18: value 324k -> 540k
- moved J7 56.4 mm to (83.8, 58.2)
- moved J4 9.55 mm to (25.5, 61.2)
- moved R2 8.89 mm to (44.7, 68.9)
- moved C4 8.89 mm to (48.8, 64.8)
- moved DEBUG_3 8.89 mm to (32.5, 71.8)
- moved DEBUG_1 8.89 mm to (38.0, 43.2)
- moved J3 8.89 mm to (26.1, 47.2)
- moved Q2 8.89 mm to (39.0, 59.8)
- moved R3 8.89 mm to (37.6, 49.2)
- moved R9 8.89 mm to (33.0, 49.2)
- moved RV1 8.89 mm to (38.7, 65.7)
- moved R_pullup1 8.89 mm to (31.5, 43.8)
- moved U1 8.89 mm to (33.0, 65.2)
- moved U4 8.89 mm to (49.7, 49.0)
- moved R17 8.89 mm to (47.2, 69.6)
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Connections:
- J7 pad 1: 12V_UNISO -> 12V_ISO
- J7 pad 2: HighVoltage- -> GND_ISO
Routing:
- net GND_ISO: track 54.7 -> 6.86 mm
- net HighVoltage-: track 141.4 -> 114.2 mm
- net 12V_ISO: track 86.9 -> 107.4 mm
- net Net-(R13-Pad2): track 6.42 -> 1.95 mm
- net Net-(DEBUG_2-A): track 7.77 -> 12.0 mm
- net Net-(Q2-D): track 16.3 -> 20.5 mm
- net Net-(R9-Pad2): track 29.3 -> 33.3 mm
- net Net-(R16-Pad2): track 1.67 -> 5.24 mm
- net Net-(DEBUG_2-K): track 26.7 -> 29.2 mm
- net Net-(R12-Pad2): track 1.67 -> 3.90 mm
- net 12V_UNISO: track 76.0 -> 77.8 mm
- net V_BIAS: track 68.7 -> 67.1 mm
- net V_IN: track 19.3 -> 20.7 mm, vias 1 -> 0
- net Net-(R14-Pad1): track 2.94 -> 1.92 mm
- net HighVoltage+: track 9.23 -> 10.2 mm
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Other:
- board text added: "+12V_ISO"
- board text removed: "+12V_UNISO"
