File: RTM/2026.2/RTM.kicad_sch (KiCad schematic)
At the start: 45 parts, among them J1 V_BIAS TEST, J2 Conn_01x02, J3 12V TEST, J4 V_IN TEST, J5 Conn_01x02, J7 Conn_01x02, Q2 NMOS, Q4 NMOS, Q5 NMOS, U1 MMSZ5245BT1G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

Commit message: Add files via upload
Parts:
- R1, R11, R12, R16, R18: value 324k -> 540k
Connections:
- net +12V: now also J7.1 (Pin_1)
- net 12V_UNISO: no longer J7.1 (Pin_1)
- net GND: no longer J7.2 (Pin_2)
- net GND_ISO: now also J7.2 (Pin_2)
Changed lines of the file:
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@@
 		)
 	)
-	(text_box "60V threshold\ndefined using \nRV1 tuned \nto 2.5k"
-		(exclude_from_sim no)
-		(at 156.21 165.1 0)
-		(size 17.78 11.43)
-		(margins 0.9525 0.9525 0.9525 0.9525)
-		(stroke
-			(width 0)
-			(type solid)
-		)
-		(fill
-			(type color)
-			(color 239 242 255 1)
-		)
-		(effects
-			(font
-				(size 1.27 1.27)
-			)
-			(justify left top)
-		)
-	)
 	(text_box "The high voltage is converted down through a voltage divider network to form V_IN. \n\nThese resistors are rated for at least 0.25W to ensure proper performance at high voltages."
 		(exclude_from_sim no)
@@
 		)
 	)
-	(global_label "12V_UNISO"
+	(global_label "12V_ISO"
 		(shape input)
 		(at 109.22 179.07 270)
@@
 		)
 		(property "Intersheetrefs" "${INTERSHEET_REFS}"
-			(at 109.22 192.3362 90)
+			(at 109.22 189.6752 90)
 			(effects
 				(font
@@
 			)
 		)
-		(property "Value" "324k"
+		(property "Value" "540k"
 			(at 102.87 130.81 90)
 			(effects
@@
 			)
 		)
-		(property "Value" "324k"
+		(property "Value" "540k"
 			(at 92.71 130.81 90)
 			(effects
@@
 			)
 		)
-		(property "Value" "324k"
+		(property "Value" "540k"
 			(at 113.03 130.81 90)
 			(effects
@@
 	)
 	(symbol
-		(lib_id "power:GND")
-		(at 113.03 179.07 0)
-		(unit 1)
-		(exclude_from_sim no)
-		(in_bom yes)
-		(on_board yes)
-		(dnp no)
-		(fields_autoplaced yes)
-		(property "Reference" "#PWR01"
-			(at 113.03 185.42 0)
-			(effects
-				(font
-					(size 1.27 1.27)
-				)
-				(hide yes)
-			)
-		)
-		(property "Value" "GND"
-			(at 113.03 184.15 0)
-			(effects
-				(font
-					(size 1.27 1.27)
-				)
-			)
-		)
-		(property "Footprint" ""
-			(at 113.03 179.07 0)
-			(effects
-				(font
-					(size 1.27 1.27)
-				)
-				(hide yes)
-			)
-		)
-		(property "Datasheet" ""
-			(at 113.03 179.07 0)
-			(effects
-				(font
-					(size 1.27 1.27)
-				)
-				(hide yes)
-			)
-		)
-		(property "Description" "Power symbol creates a global label with name \"GND\" , ground"
-			(at 113.03 179.07 0)
-			(effects
-				(font
-					(size 1.27 1.27)
-				)
-				(hide yes)
-			)
-		)
-		(pin "1"
-		)
-		(instances
-			(project "TS_READY_TO_MOVE (1)"
-				(path "/ec2b8551-75c2-4864-b31d-b681332831c2"
-					(reference "#PWR01")
-					(unit 1)
-				)
-			)
-		)
-	)
-	(symbol
 		(lib_id "Device:R_US")
 		(at 80.01 153.67 90)
@@
 			)
 		)
-		(property "Value" "324k"
+		(property "Value" "540k"
 			(at 80.01 130.81 90)
 			(effects
@@
 			)
 		)
-		(property "Value" "324k"
+		(property "Value" "540k"
 			(at 66.04 130.81 90)
 			(effects
@@
 					(unit 1)
 				)
+			)
+		)
+	)
+	(symbol
+		(lib_id "power:GNDPWR")
+		(at 113.03 179.07 0)
+		(unit 1)
+		(exclude_from_sim no)
+		(in_bom yes)
+		(on_board yes)
+		(dnp no)
+		(fields_autoplaced yes)
+		(property "Reference" "#PWR018"
+			(at 113.03 184.15 0)
+			(effects
+				(font
+					(size 1.27 1.27)
+				)
+				(hide yes)
+			)
+		)
+		(property "Value" "GND_ISO"
+			(at 112.903 182.88 0)
+			(effects
+				(font
+					(size 1.27 1.27)
+				)
+			)
+		)
+		(property "Footprint" ""
+			(at 113.03 180.34 0)
+			(effects
+				(font
+					(size 1.27 1.27)
+				)
+				(hide yes)
+			)
+		)
+		(property "Datasheet" ""
+			(at 113.03 180.34 0)
+			(effects
+				(font
+					(size 1.27 1.27)
+				)
+				(hide yes)
+			)
+		)
+		(property "Description" "Power symbol creates a global label with name \"GNDPWR\" , global ground"
+			(at 113.03 179.07 0)
+			(effects
+				(font
+					(size 1.27 1.27)
+				)
+				(hide yes)
+			)
+		)
+		(pin "1"
+		)
+		(instances
+			(project "RTM"
+				(path "/ec2b8551-75c2-4864-b31d-b681332831c2"
+					(reference "#PWR018")
+					(unit 1)
+				)
