File: RTM/2026.2/RTM_2026.2.kicad_sch (KiCad schematic)
At the start: 45 parts, among them J1 V_BIAS TEST, J2 Conn_01x02, J3 12V TEST, J4 V_IN TEST, J5 Conn_01x02, J7 Conn_01x02, Q2 NMOS, Q4 NMOS, Q5 NMOS, U1 MMSZ5245BT1G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

Commit message: Changed all NMOS to GDS
Parts:
- removed Q2, Q4, Q5: NMOS, Package_TO_SOT_THT:TO-220-3_Vertical, symbol Simulation_SPICE:NMOS
- added Q2, Q4, Q5: NMOS, Package_TO_SOT_THT:TO-220-3_Vertical, symbol Transistor_FET:Q_NMOS_GDS
Connections:
- net GND: now also Q2.3 (S)
- net GND_ISO: now also Q4.3 (S), Q5.3 (S)
- net at DEBUG_1.1 (K), R_pullup1.2, U4.1 (OUT): now also Q2.1 (G)
- net at R4.2, U3.4 (R): now also Q4.2 (D)
- net at DEBUG_2.1 (K), R10.2, U2.5: now also Q4.1 (G)
- net at U3.3 (Q): now also Q5.1 (G)
- net at U2.2: now also Q2.2 (D)
- net at J2.2 (Pin_2), R7.2: now also Q5.2 (D)
