File: BSPD/2026.2/bspd_2026/bspd.kicad_pcb (KiCad board)
At the start: 2 copper layers, 80 x 70 mm, 69 parts, among them J1 Conn_01x02, J2 Conn_01x02, J3 Conn_01x02, J4 Conn_01x02, Q1 IRLIZ44N NMOS, U1 40106, U2 4081 AND Gate, U3 LM393, U4 LM393, U5 4071 OR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

Commit message: bspd v3 plus documentation
Parts:
- added J5: T2M-105-01-X-D-TH-DS, T2M_105:SAMTEC_T2M-105-01-X-D-TH-DS, F.Cu at (213.0, 78.0)
- U5: value 4071 OR -> 4071 4 Channel 2 Input OR gate
- moved H2 10.0 mm to (213.0, 47.0)
- moved H3 10.0 mm to (213.0, 107.0)
Routing:
- net +12V: track 293.5 -> 295.0 mm
Other:
- board size 80 x 70 mm -> 90 x 70 mm
