File: BSPD/2026.2/bspd_2026/bspd.kicad_sch (KiCad schematic)
At the start: 71 parts, among them J1 Conn_01x02, J2 Conn_01x02, J3 Conn_01x02, J4 Conn_01x02, Q1 IRLIZ44N NMOS, U1 40106, U2 4081 AND Gate, U3 LM393, U4 LM393, U5 4071 4 Channel 2 Input OR gate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

Commit message: bspd v3 plus documentation
Parts:
- removed D3: 1N47xxA, Diode_THT:D_DO-41_SOD81_P10.16mm_Horizontal, symbol Diode:1N47xxA
- removed R20: 50, Resistor_SMD:R_0603_1608Metric, symbol Device:R
- added J5: T2M-105-01-X-D-TH-DS, T2M_105:SAMTEC_T2M-105-01-X-D-TH-DS, symbol T2M-105-01-X-D-TH-DS:T2M-105-01-X-D-TH-DS
Connections:
- net +12V: now also J5.01, J5.03
- net BRAKE: now also J5.07
- net BSPD_FAULT: now also J5.09
- net GND: now also J5.02, J5.04, J5.06, J5.08, J5.10
- net PEDAL: now also J5.05
