File: TSSI/2026.3/TSSI2026.3/TSSI2026.3.kicad_pcb (KiCad board)
At the start: 2 copper layers, 40 x 39.5 mm, 26 parts, among them J1 Conn_02x02, J2 Conn_01x02, Q1 IRLZ34N, Q2 IRLZ34N, Q3 IRLZ34N, T555 Test555, U1 LM555xN, U3 IRLZ34N

Commit message: Add Logo again
Parts:
- added G***: LOGO, LOGO, F.Cu at (51.0, 89.0)
