File: BSPD/2026.3/bspd_2026/bspd.kicad_pcb (KiCad board)
At the start: 2 copper layers, 90 x 70 mm, 75 parts, among them J1 T2M-105-01-X-D-TH-DS, J2 39-30-6068, Q1 IRLIZ44N NMOS, U1 LM393, U2 4071 4 Channel 2 Input OR gate, U3 LM393, U4 LM393, U5 4081 AND Gate, U6 40106

Commit message: fixed comparator pinouts and pcb layout
Parts:
- U6: value 40106 -> 40106 Inverter
Connections:
- U1 pad 2: SHORT_CIRCUIT -> BRAKE
- U1 pad 3: BRAKE -> SHORT_CIRCUIT
- U4 pad 2: SHORT_CIRCUIT -> CURRENT
- U4 pad 3: CURRENT -> SHORT_CIRCUIT
Routing:
- net BRAKE: track 74.6 -> 75.7 mm
