File: SafetyBoard/CCMIO.kicad_sch (KiCad schematic)
At the start: 24 parts, among them J12 RTD B, J13 Brakelight, J14 SHOCK/WHEEL SNSR, J15 TO CCM, J16 FOOTWELL, J17 Conn_01x04_Pin

Commit message: hopefully this lets avadi pull
Parts:
- removed J15: TO CCM, 1MyCustomLibrary:MOLEX_39281123, symbol 39281123:39281123
- added J17: SHOCK/WHEEL SNSR, footprints:12pSTminifit, symbol 39281123:39281123
- J15: renamed from J14; footprint 1MyCustomLibrary:MOLEX_39281123 -> footprints:12pSTminifit
- J16: value FOOTWELL -> SHOCK/WHEEL SNSR; footprint 1MyCustomLibrary:MOLEX_39281123 -> footprints:12pSTminifit
- renumbered C16 to C18, C17 to C19, C20 to C26, C22 to C28, C23 to C29, C24 to C30, C25 to C31, J12 to J13, J13 to J14, J17 to J18, R48 to R49, R49 to R50, R50 to R51, R51 to R52, R52 to R54, R54 to R56, R55 to R57, R56 to R58, R57 to R59
Connections:
- net 12V: now also J16.3
- net 24V: now also J16.4
- net 5V: now also J16.6, J17.10, J17.7; no longer J16.10, J16.7
- net APPS1 IN: now also J17.3; no longer J16.3
- net APPS1 OUT: now also J16.11
- net APPS2 IN: now also J17.6; no longer J16.6
- net APPS2 OUT: now also J16.12
- net BPS1 IN: now also J17.12; no longer J16.12
- net BPS1 OUT: now also J16.9
- net BPS2 IN: now also J17.9; no longer J16.9
- net BPS2 OUT: now also J16.10
- net Brakelight: now also J16.2
- net CCM3v3: now also J16.8, J17.1, J17.4; no longer J16.1, J16.4
- net CCMGND: now also J16.7, J17.11, J17.2, J17.5, J17.8; no longer J16.11, J16.2, J16.5, J16.8
- net GND: now also J16.1
- net RTDB: now also J16.5

Commit message: rough layout done
Parts:
- removed J16, J17: SHOCK/WHEEL SNSR, footprints:12pSTminifit, symbol 39281123:39281123
- added J16: footwell, footprints:14pSTminifit, symbol 14pSTminifit:39299142
- added J19: 39306207, footprints:20pSTminfit, symbol 20pSTminifit:39306207
- J18: value Conn_01x04_Pin -> AMP
Connections:
- net BPS1_OUT is gone; now on net BPS1 OUT: R51.2
- net 24V: now also J19.4
- net 5V: now also J15.2, J15.7, J15.8, J16.1, J16.8; no longer J15.4, J15.5, J15.6
- net APPS1 IN: now also J16.5
- net APPS1 OUT: now also J19.8
- net APPS2 IN: now also J16.6
- net APPS2 OUT: now also J19.9
- net BPS1 OUT: now also J19.5
- net BPS2 IN: now also J16.3
- net BPS2 OUT: now also J19.6
- net Brakelight: now also J19.20
- net CCM fdbk: now also J19.2
- net CCM3v3: now also J16.11, J19.7
- net CCMGND: now also J15.4, J15.5, J15.6, J16.10, J16.12, J16.13, J16.9, J19.12; no longer J15.10, J15.12, J15.8
- net Speaker IN: now also J19.3
- net TSSI BYP: now also J19.1
- net Wheel/Shock1 IN: now also J15.9; no longer J15.7
- net Wheel/Shock1 OUT: now also J19.14
- net Wheel/Shock2 IN: now also J15.10; no longer J15.9
- net Wheel/Shock2 OUT: now also J19.15
- net Wheel/Shock3 OUT: now also J19.16
- net Wheel/Shock4 IN: now also J15.12; no longer J15.2
- net Wheel/Shock4 OUT: now also J19.17
- net BPS1 IN renamed BPS 1
- net BPS 1: now also J16.2
