File: SafetyBoard/CCMIO.kicad_sch (KiCad schematic)
At the start: 24 parts, among them J14 footwell, J15 RTD B, J16 Brakelight, J17 SHOCK/WHEEL SNSR, J18 39306207, J19 AMP

Commit message: updates I think
Connections:
- net 5V: now also J14.14, J14.7; no longer J14.1, J14.8
- net APPS1 IN: now also J14.10; no longer J14.5
- net APPS2 IN: now also J14.9; no longer J14.6
- net BPS1 IN: now also J14.13; no longer J14.2
- net BPS2 IN: now also J14.12; no longer J14.3
- net CCMGND: now also J14.2, J14.3, J14.5, J14.6; no longer J14.10, J14.12, J14.13, J14.9
- no-connect marks 3 -> 1
Changed lines of the file:
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@@
 	(paper "A4")
 	(no_connect
-		(at 52.07 76.2)
-	)
-	(no_connect
 		(at 181.61 95.504)
 	)
-	(no_connect
-		(at 52.07 58.42)
-	)
 	(wire
 		(pts
@@
 		)
 	)
-	(label "APPS2 IN"
-		(at 52.07 55.88 180)
+	(label "5V"
+		(at 52.07 76.2 180)
 		(effects
 			(font
@@
 		)
 	)
+	(label "CCMGND"
+		(at 52.07 48.26 180)
+		(effects
+			(font
+				(size 1.27 1.27)
+			)
+			(justify right bottom)
+		)
+	)
 	(label "BPS2 IN"
 		(at 105.664 147.32 0)
@@
 		)
 	)
-	(label "BPS2 IN"
-		(at 52.07 48.26 180)
+	(label "APPS2 IN"
+		(at 52.07 63.5 180)
 		(effects
 			(font
@@
 		)
 	)
+	(label "5V"
+		(at 52.07 58.42 180)
+		(effects
+			(font
+				(size 1.27 1.27)
+			)
+			(justify right bottom)
+		)
+	)
 	(label "Wheel{slash}Shock4 IN"
 		(at 98.298 35.56 180)
@@
 		)
 	)
-	(label "BPS1 IN"
-		(at 52.07 45.72 180)
-		(effects
-			(font
-				(size 1.27 1.27)
-			)
-			(justify right bottom)
-		)
-	)
-	(label "CCMGND"
-		(at 52.07 66.04 180)
-		(effects
-			(font
-				(size 1.27 1.27)
-			)
-			(justify right bottom)
-		)
-	)
 	(label "CCMGND"
 		(at 252.476 136.906 180)
@@
 	)
 	(label "CCMGND"
+		(at 52.07 45.72 180)
+		(effects
+			(font
+				(size 1.27 1.27)
+			)
+			(justify right bottom)
+		)
+	)
+	(label "CCMGND"
 		(at 55.88 181.61 180)
 		(effects
@@
 		)
 	)
+	(label "BPS2 IN"
+		(at 52.07 71.12 180)
+		(effects
+			(font
+				(size 1.27 1.27)
+			)
+			(justify right bottom)
+		)
+	)
+	(label "BPS1 IN"
+		(at 52.07 73.66 180)
+		(effects
+			(font
+				(size 1.27 1.27)
+			)
+			(justify right bottom)
+		)
+	)
+	(label "APPS1 IN"
+		(at 52.07 66.04 180)
+		(effects
+			(font
+				(size 1.27 1.27)
+			)
+			(justify right bottom)
+		)
+	)
+	(label "CCMGND"
+		(at 52.07 53.34 180)
+		(effects
+			(font
+				(size 1.27 1.27)
+			)
+			(justify right bottom)
+		)
+	)
 	(label "CCMGND"
 		(at 123.698 35.56 0)
@@
 		)
 	)
-	(label "5V"
-		(at 52.07 60.96 180)
-		(effects
-			(font
-				(size 1.27 1.27)
-			)
-			(justify right bottom)
-		)
-	)
 	(label "APPS2 OUT"
 		(at 181.61 72.644 180)
@@
 		)
 	)
-	(label "5V"
-		(at 52.07 43.18 180)
-		(effects
-			(font
-				(size 1.27 1.27)
-			)
-			(justify right bottom)
-		)
-	)
 	(label "RTDB"
 		(at 181.61 77.724 180)
@@
 		)
 	)
-	(label "APPS1 IN"
-		(at 52.07 53.34 180)
-		(effects
-			(font
-				(size 1.27 1.27)
-			)
-			(justify right bottom)
-		)
-	)
-	(label "CCMGND"
-		(at 52.07 63.5 180)
+	(label "CCMGND"
+		(at 52.07 55.88 180)
 		(effects
 			(font
@@
 	)
 	(label "CCMGND"
-		(at 52.07 73.66 180)
-		(effects
-			(font
-				(size 1.27 1.27)
-			)
-			(justify right bottom)
-		)
-	)
-	(label "CCMGND"
 		(at 225.298 161.29 0)
 		(effects
@@
 		)
 	)
-	(label "CCMGND"
-		(at 52.07 71.12 180)
-		(effects
-			(font
-				(size 1.27 1.27)
-			)
-			(justify right bottom)
-		)
-	)
