File: SafetyBoard/SafetyBoard.kicad_pcb (KiCad board)
At the start: 2 copper layers, 177 parts, among them J10 Suspension_Linear_Pot3, J11 Suspension_Linear_Pot4, J12 12V_EXP1, J13 12V_EXP3, J14 12V_EXP2, J15 3V3_EXP, J16 RTM, J17 Throttle_Sensor, J18 Wheel_Sensor1, J19 Wheel_Sensor2, J20 24V_IN, J21 Back_Of_Car_12V, J22 24V_EXP1, J23 24V_OUT, J24 RasPI_5V, J25 EXP1_5V, J26 BSPD, J27 LATCH, J28 TSSI, J29 CCM_Faults, J30 CCM_12V, J31 LATCH_12V, J8 Suspension_Linear_Pot1, J9 Suspension_Linear_Pot2, Q1 IRLIZ44N NMOS, Q4 PMOS IRF9540, Q5 PMOS IRF9540, Q6 PMOS IRF9540, SW1 SW_Push, SW2 SW_Push, SW3 SW_Push, T1 Test555, U1 40106 Inverter, U10 AP63200WU, U12 ACS711xLCTR-12AB, U2 4081 AND Gate, U3 LM393, U4 LM393, U5 4071 4 Channel 2 Input OR gate, U6 LM393, U7 LM555xN, U9 LT1084-5.0

Commit message: day 2 grind
Parts:
- removed D14: 1.5SMCxxA, Diode_SMD:D_SMC
- removed F10, F11, F12, F7, F8: 500mA, 0footprints:FUSE_3522-2
- removed F9: 10A, 0footprints:FUSE_3522-2
- removed H13, H14, H15, H16: MountingHole M3, MountingHole:MountingHole_3.2mm_M3_Pad
- removed J10: Suspension_Linear_Pot3, 0footprints:Molex_Mini-Fit_Jr_5566-04A_2x02_P4.20mm_Vertical
- removed J11: Suspension_Linear_Pot4, 0footprints:Molex_Mini-Fit_Jr_5566-04A_2x02_P4.20mm_Vertical
- removed J14: 12V_EXP2, 0footprints:Molex_Mini-Fit_Jr_5566-02A_2x01_P4.20mm_Vertical
- removed J15: 3V3_EXP, 0footprints:Molex_Mini-Fit_Jr_5566-02A_2x01_P4.20mm_Vertical
- removed J16: RTM, 0footprints:Molex_Mini-Fit_Jr_5566-02A_2x01_P4.20mm_Vertical
- removed J19: Wheel_Sensor2, 0footprints:Molex_Mini-Fit_Jr_5566-04A_2x02_P4.20mm_Vertical
- removed J20: 24V_IN, 0footprints:Molex_Mini-Fit_Jr_5566-02A_2x01_P4.20mm_Vertical
- removed J21: Back_Of_Car_12V, 0footprints:Molex_Mini-Fit_Jr_5566-02A_2x01_P4.20mm_Vertical
- removed J22: 24V_EXP1, 0footprints:Molex_Mini-Fit_Jr_5566-02A_2x01_P4.20mm_Vertical
- removed J23: 24V_OUT, 0footprints:Molex_Mini-Fit_Jr_5566-02A_2x01_P4.20mm_Vertical
- removed J24: RasPI_5V, 0footprints:Molex_Mini-Fit_Jr_5566-02A_2x01_P4.20mm_Vertical
- removed J25: EXP1_5V, 0footprints:Molex_Mini-Fit_Jr_5566-02A_2x01_P4.20mm_Vertical
- removed J26: BSPD, 0footprints:Molex_Mini-Fit_Jr_5566-06A_2x03_P4.20mm_Vertical
- removed J27: LATCH, 0footprints:Molex_Mini-Fit_Jr_5566-08A_2x04_P4.20mm_Vertical
- removed J28: TSSI, 0footprints:Molex_Mini-Fit_Jr_5566-04A_2x02_P4.20mm_Vertical
- removed J29: CCM_Faults, 0footprints:Molex_Mini-Fit_Jr_5566-10A_2x05_P4.20mm_Vertical
- removed J30: CCM_12V, 0footprints:Molex_Mini-Fit_Jr_5566-02A_2x01_P4.20mm_Vertical
- removed J31: LATCH_12V, 0footprints:Molex_Mini-Fit_Jr_5566-02A_2x01_P4.20mm_Vertical
- removed L1: 10uH, Inductor_SMD:L_0603_1608Metric_Pad1.05x0.95mm_HandSolder
- removed the R47 at (143.0, 134.0)
- removed U12: ACS711xLCTR-12AB, Package_SO:SOIC-8_3.9x4.9mm_P1.27mm
- added C1: 0.1u, Capacitor_SMD:C_0603_1608Metric, F.Cu at (46.2, 241.8)
- added C10: 1n, Capacitor_SMD:C_0603_1608Metric, F.Cu at (71.4, 286.3)
- added C15: 1u, Capacitor_SMD:C_0805_2012Metric, F.Cu at (311.3, 127.6)
- added C18: 330uF, Capacitor_SMD:C_2220_5750Metric_Pad1.97x5.40mm_HandSolder, F.Cu at (493.1, -8.11)
- added C2: 0.1u, Capacitor_SMD:C_0603_1608Metric, F.Cu at (66.9, 242.3)
- added C20: 10n, Capacitor_SMD:C_0805_2012Metric, F.Cu at (255.3, 83.8)
- added C22: 100n, Capacitor_SMD:C_0805_2012Metric, F.Cu at (255.3, 89.8)
- added C24: 100n, Capacitor_SMD:C_0805_2012Metric, F.Cu at (255.3, 92.8)
- added C25: 100n, Capacitor_SMD:C_0805_2012Metric, F.Cu at (255.3, 86.8)
- added C26: 330uF, Capacitor_SMD:C_2220_5750Metric_Pad1.97x5.40mm_HandSolder, F.Cu at (415.1, -56.3)
- added C27: 330uF, Capacitor_SMD:C_2220_5750Metric_Pad1.97x5.40mm_HandSolder, F.Cu at (415.1, -49.3)
- added C28: 22uF, Capacitor_SMD:C_0805_2012Metric, F.Cu at (399.6, -43.3)
- added C29: 22uF, Capacitor_SMD:C_0805_2012Metric, F.Cu at (399.6, -40.3)
- added C3: 0.1u, Capacitor_SMD:C_0603_1608Metric, F.Cu at (47.2, 257.8)
- added C30: 10u, Capacitor_SMD:C_0805_2012Metric, F.Cu at (399.6, -37.3)
- added C31: 330uF, Capacitor_SMD:C_2220_5750Metric_Pad1.97x5.40mm_HandSolder, F.Cu at (415.1, -42.4)
- added C4: 0.1u, Capacitor_SMD:C_0603_1608Metric, F.Cu at (66.4, 265.8)
- added C5: 0.1u, Capacitor_SMD:C_0603_1608Metric, F.Cu at (46.4, 274.8)
- added C6: 0.1u, Capacitor_SMD:C_0603_1608Metric, F.Cu at (87.7, 265.0)
- added C7: 3.3u, Capacitor_SMD:C_0603_1608Metric, F.Cu at (72.4, 271.8)
- added C8: 10u, Capacitor_SMD:C_0603_1608Metric, F.Cu at (34.2, 289.3)
- added C9: 1n, Capacitor_SMD:C_0603_1608Metric, F.Cu at (34.2, 295.1)
- added D1: D, Diode_SMD:D_0603_1608Metric, F.Cu at (69.2, 266.6)
- added D2: D, Diode_SMD:D_0603_1608Metric, F.Cu at (36.7, 289.3)
- added FL1: RGF48040A-001, DCDCfootprints:EMI Filter RGF48040A001, F.Cu at (459.5, -28.2)
- added H1: MH, MountingHole:MountingHole_3mm, F.Cu at (14.2, 235.3)
- added H2: MH, MountingHole:MountingHole_3mm, F.Cu at (94.2, 235.3)
- added H3: MH, MountingHole:MountingHole_3mm, F.Cu at (14.2, 295.3)
- added H4: MH, MountingHole:MountingHole_3mm, F.Cu at (94.2, 295.3)
- added J1: T2M-105-01-X-D-TH-DS, T2M_105:SAMTEC_T2M-105-01-X-D-TH-DS, F.Cu at (94.6, 269.8)
- added J1: ESTOP/SDC switch, 0footprints:Molex_Mini-Fit_Jr_5566-02A_2x01_P4.20mm_Vertical, F.Cu at (238.9, 104.6)
- added J2: SDC OUT, 0footprints:Molex_Mini-Fit_Jr_5566-02A_2x01_P4.20mm_Vertical, F.Cu at (246.4, 104.6)
- added J2: 39-30-6068, 39-30:39-30-606Y, F.Cu at (49.0, 290.3)
- added J3: SDC OUT, 0footprints:Molex_Mini-Fit_Jr_5566-02A_2x01_P4.20mm_Vertical, F.Cu at (311.5, 38.9)
- added J4: ACCU, 0footprints:Molex_Mini-Fit_Jr_5566-04A_2x02_P4.20mm_Vertical, F.Cu at (243.1, 91.5)
- added J5: BSPD, 0footprints:Molex_Mini-Fit_Jr_5566-06A_2x03_P4.20mm_Vertical, F.Cu at (223.1, 104.6)
- added J6: LATCH, 0footprints:Molex_Mini-Fit_Jr_5566-08A_2x04_P4.20mm_Vertical, F.Cu at (229.4, 94.3)
- added J7: ACCU, 0footprints:Molex_Mini-Fit_Jr_5566-04A_2x02_P4.20mm_Vertical, F.Cu at (311.5, 52.0)
- added LED1: APTD2012LSYCK, SMALL_LED:LEDC2012X105N, F.Cu at (49.0, 268.2)
- added LED2: APTD2012LSYCK, SMALL_LED:LEDC2012X105N, F.Cu at (67.8, 281.5)
- added LED3: APTD2012LSYCK, SMALL_LED:LEDC2012X105N, F.Cu at (70.8, 275.6)
- added PS1: I7A24080A033V-0C3-R, DCDCfootprints:24V DCDC I7A24080A033V0C3R, F.Cu at (455.6, -2.73)
- added Q1: IRLIZ44N NMOS, Package_TO_SOT_THT:TO-220F-3_Vertical, F.Cu at (75.9, 249.3)
- added R1: 20k, Resistor_SMD:R_0603_1608Metric, F.Cu at (29.2, 241.8)
- added R10: 10K, Resistor_SMD:R_0603_1608Metric, F.Cu at (21.2, 273.8)
- added R11: 20k, Resistor_SMD:R_0603_1608Metric, F.Cu at (31.0, 258.0)
- added R12: 20k, Resistor_SMD:R_0603_1608Metric, F.Cu at (46.7, 276.8)
- added R13: 20k, Resistor_SMD:R_0603_1608Metric, F.Cu at (47.4, 260.3)
- added R14: 120k, Resistor_SMD:R_0603_1608Metric, F.Cu at (72.4, 265.8)
- added R15: 1k, Resistor_SMD:R_0603_1608Metric, F.Cu at (72.4, 268.3)
- added R16: 10K, Resistor_SMD:R_0603_1608Metric, F.Cu at (20.7, 286.8)
- added R17: 10K, Resistor_SMD:R_0603_1608Metric, F.Cu at (20.5, 281.8)
- added R18: 500k, Resistor_SMD:R_0603_1608Metric, F.Cu at (38.9, 295.1)
- added R19: 1k, Resistor_SMD:R_0603_1608Metric, F.Cu at (36.5, 295.1)
- added R2: 10K, Resistor_SMD:R_0603_1608Metric, F.Cu at (21.0, 248.3)
- added R20: 1k, Resistor_SMD:R_0603_1608Metric, F.Cu at (67.8, 286.3)
- added R21: 500k, Resistor_SMD:R_0603_1608Metric, F.Cu at (67.7, 283.8)
- added R22: 10k, Resistor_SMD:R_0603_1608Metric, F.Cu at (49.1, 271.7)
- added R23: 10k, Resistor_SMD:R_0603_1608Metric, F.Cu at (67.8, 273.3)
- added R24: 10k, Resistor_SMD:R_0603_1608Metric, F.Cu at (66.8, 279.0)
- added R3: 10K, Resistor_SMD:R_0603_1608Metric, F.Cu at (21.0, 243.3)
- added R4: 20k, Resistor_SMD:R_0603_1608Metric, F.Cu at (47.5, 244.3)
- added R5: 10k, Resistor_SMD:R_0603_1608Metric, F.Cu at (74.8, 244.6)
- added R51: 1.5K, Resistor_SMD:R_0805_2012Metric, F.Cu at (315.8, 133.5)
- added R52: 1k, Resistor_SMD:R_0805_2012Metric, F.Cu at (259.7, 83.8)
- added R53: 1.05k, Resistor_SMD:R_0805_2012Metric, F.Cu at (419.5, -24.5)
- added R54: 1k, Resistor_SMD:R_0805_2012Metric, F.Cu at (259.7, 89.7)
- added R55: 1k, Resistor_SMD:R_0805_2012Metric, F.Cu at (259.7, 95.6)
- added R56: 1k, Resistor_SMD:R_0805_2012Metric, F.Cu at (259.7, 92.6)
- added R57: 1k, Resistor_SMD:R_0805_2012Metric, F.Cu at (259.7, 86.7)
- added R58: 1.47k, Resistor_SMD:R_0805_2012Metric_Pad1.20x1.40mm_HandSolder, F.Cu at (399.8, -34.3)
- added R6: 10K, Resistor_SMD:R_0603_1608Metric, F.Cu at (21.2, 256.3)
- added R7: 10K, Resistor_SMD:R_0603_1608Metric, F.Cu at (21.2, 261.3)
- added R8: 10K, Resistor_SMD:R_0603_1608Metric, F.Cu at (21.0, 268.8)
- added R9: 20k, Resistor_SMD:R_0603_1608Metric, F.Cu at (30.4, 274.3)
- added R_Bypass1: 0, Resistor_SMD:R_0603_1608Metric, F.Cu at (77.7, 287.9)
- added R_Bypass2: 0, Resistor_SMD:R_0603_1608Metric, F.Cu at (83.2, 287.9)
- added TP1: B_SHORT, TestPoint:TestPoint_Pad_D2.5mm, F.Cu at (30.2, 237.3)
- added TP10: SC, TestPoint:TestPoint_Pad_D2.5mm, F.Cu at (25.7, 258.8)
- added TP11: P_SHORT, TestPoint:TestPoint_Pad_D2.5mm, F.Cu at (36.2, 270.8)
- added TP12: P_APPLIED, TestPoint:TestPoint_Pad_D2.5mm, F.Cu at (48.7, 263.3)
- added TP13: BSPD_FAULT, TestPoint:TestPoint_Pad_D2.5mm, F.Cu at (80.1, 259.6)
- added TP14: PEDAL, TestPoint:TestPoint_Pad_D2.5mm, F.Cu at (30.8, 294.3)
- added TP15: PEDAL_TH, TestPoint:TestPoint_Pad_D2.5mm, F.Cu at (25.2, 284.3)
- added TP16: BRAKE, TestPoint:TestPoint_Pad_D2.5mm, F.Cu at (52.7, 284.2)
- added TP17: P_OPEN, TestPoint:TestPoint_Pad_D2.5mm, F.Cu at (47.2, 284.3)
- added TP2: OC, TestPoint:TestPoint_Pad_D2.5mm, F.Cu at (25.2, 245.8)
- added TP3: B_OPEN, TestPoint:TestPoint_Pad_D2.5mm, F.Cu at (47.2, 248.8)
- added TP4: P_ERROR, TestPoint:TestPoint_Pad_D2.5mm, F.Cu at (64.7, 238.3)
- added TP5: FAULT_SENSED, TestPoint:TestPoint_Pad_D2.5mm, F.Cu at (69.9, 249.8)
- added TP6: B_ERROR, TestPoint:TestPoint_Pad_D2.5mm, F.Cu at (60.7, 238.3)
- added TP7: BOTH_ON, TestPoint:TestPoint_Pad_D2.5mm, F.Cu at (67.2, 246.8)
- added TP8: BRAKE_TH, TestPoint:TestPoint_Pad_D2.5mm, F.Cu at (25.2, 271.3)
- added TP9: B_APPLIED, TestPoint:TestPoint_Pad_D2.5mm, F.Cu at (29.7, 261.3)
- added U1: LM393, Package_DIP:DIP-8_W7.62mm_Socket, F.Cu at (34.9, 242.0)
- added U2: 4071 4 Channel 2 Input OR gate, Package_DIP:DIP-14_W7.62mm_Socket, F.Cu at (55.6, 242.2)
- added U3: LM393, Package_DIP:DIP-8_W7.62mm_Socket, F.Cu at (34.9, 258.0)
- added U4: LM393, Package_DIP:DIP-8_W7.62mm_Socket, F.Cu at (34.9, 274.5)
- added U5: 4081 AND Gate, Package_DIP:DIP-14_W7.62mm_Socket, F.Cu at (55.4, 265.7)
- added U6: 40106 Inverter, Package_DIP:DIP-14_W7.62mm_Socket, F.Cu at (77.1, 265.8)
- added VR1: 3296Y-11-103LF, Potentiometer_THT:Potentiometer_Bourns_3296Y_Vertical, F.Cu at (12.2, 243.3)
- added VR2: 3296Y-11-103LF, Potentiometer_THT:Potentiometer_Bourns_3296Y_Vertical, F.Cu at (12.2, 256.2)
- added VR3: 3296Y-11-103LF, Potentiometer_THT:Potentiometer_Bourns_3296Y_Vertical, F.Cu at (12.2, 268.8)
- added VR4: 3296Y-11-103LF, Potentiometer_THT:Potentiometer_Bourns_3296Y_Vertical, F.Cu at (12.2, 281.8)
- C14: value 100nF -> 1u; footprint Capacitor_SMD:C_0603_1608Metric_Pad1.08x0.95mm_HandSolder -> Capacitor_SMD:C_0805_2012Metric
- C16: value 10uF -> 1u; footprint Capacitor_SMD:C_0603_1608Metric_Pad1.08x0.95mm_HandSolder -> Capacitor_SMD:C_0805_2012Metric
- C17: value 56pF -> 1u; footprint Capacitor_SMD:C_0603_1608Metric_Pad1.08x0.95mm_HandSolder -> Capacitor_SMD:C_0805_2012Metric
- C19, C21: footprint Capacitor_SMD:C_0603_1608Metric_Pad1.08x0.95mm_HandSolder -> Capacitor_SMD:C_0805_2012Metric
- C23: value 100nF -> 100n; footprint Capacitor_SMD:C_0603_1608Metric_Pad1.08x0.95mm_HandSolder -> Capacitor_SMD:C_0805_2012Metric
- F1, F2, F3, F4, F5, F6: value 500mA -> ~
- J12: value 12V_EXP1 -> RTD B
- J13: value 12V_EXP3 -> Brakelight
- J17: value Throttle_Sensor -> Conn_01x04_Pin; footprint 0footprints:Molex_Mini-Fit_Jr_5566-06A_2x03_P4.20mm_Vertical -> footprints:AmpBoard
- J18: value Wheel_Sensor1 -> 614004135023; footprint 0footprints:Molex_Mini-Fit_Jr_5566-04A_2x02_P4.20mm_Vertical -> footprints:614004135023
- J8: value Suspension_Linear_Pot1 -> Current Sensor
- J9: value Suspension_Linear_Pot2 -> TSSI
- R48: value 18k -> 1.5K; footprint Resistor_SMD:R_0603_1608Metric_Pad0.98x0.95mm_HandSolder -> Resistor_SMD:R_0805_2012Metric
- R49, R50: value 10K -> 1.5K; footprint Resistor_SMD:R_1206_3216Metric -> Resistor_SMD:R_0805_2012Metric
- U10: value AP63200WU -> OKX-T/5-D12N-C; footprint Package_TO_SOT_SMD:TSOT-23-6 -> footprints:12v5vDCDC
- moved C19 310.0 mm to (415.1, -24.4)
- moved C21 309.7 mm to (415.1, -21.4)
- moved U10 309.4 mm to (415.2, -32.9)
- moved J18 230.2 mm to (392.4, -49.2)
- moved H7 218.0 mm to (130.8, 352.4)
- moved C1 218.0 mm to (150.0, 272.7)
- moved C10 218.0 mm to (154.1, 272.7)
- moved C12 218.0 mm to (141.4, 355.2)
- moved C13 218.0 mm to (141.4, 358.2)
- moved C2 218.0 mm to (150.0, 275.2)
- moved C3 218.0 mm to (150.0, 277.7)
- moved C7 218.0 mm to (150.0, 287.7)
- moved C8 218.0 mm to (150.0, 290.2)
- moved C9 218.0 mm to (150.0, 292.7)
- moved D2 218.0 mm to (177.7, 275.3)
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- renumbered R25 to R26, R26 to R27, R27 to R28, R28 to R29, R29 to R30, R30 to R31, R31 to R32, R32 to R33, R33 to R34, R34 to R35, R35 to R36, R36 to R37, R37 to R38, R38 to R39, R39 to R40, R40 to R41, R41 to R42, R42 to R43, R43 to R44, R44 to R45, R45 to R46, R46 to R47, U9 to U3, U3 to U4, U4 to U5, U5 to U6, U6 to U7, U7 to U8
Connections:
- net /LATCH/BMS_FAULT renamed /BMS FAULT
- net /TSSI/CCMSensorFeedBack renamed /CCM Helper/CCM fdbk
- C14 pad 1: /PDB/SW -> /CCM Helper/APPS2 IN
- C14 pad 2: /PDB/BST -> /CCM Helper/CCMGND
- C16 pad 1: /PDB/BUCK_IN -> /CCM Helper/BPS1 IN
- C16 pad 2: GND -> /CCM Helper/CCMGND
- C17 pad 1: 12V -> /CCM Helper/BPS2 IN
- C17 pad 2: /PDB/FB -> /CCM Helper/CCMGND
- C19 pad 1: 12V -> Net-(FL1-VOUT(+)_)
- C21 pad 1: 12V -> 12V_OUT
- C23 pad 1: GND -> /CCM Helper/Wheel/Shock2 IN
- C23 pad 2: 3.3V -> /CCM Helper/CCMGND
- D4 pad 2: unconnected-(D4-A-Pad2) -> Net-(D4-A)
- F1 pad 1: /PDB/Fuse_EXP1_12V -> +12V
- F1 pad 2: 12V -> /12V
- F2 pad 1: /PDB/Fuse_EXP3_12V -> /12V_2
- F2 pad 2: 12V -> /12V
- F3 pad 1: /PDB/Fuse_EXP2_12V -> /CCM Helper/12V
- F3 pad 2: 12V -> /12V
- F4 pad 1: /PDB/Fuse_EXP_3V3 -> /CCM Helper/24V
- F4 pad 2: 3.3V -> /24V
- F5 pad 1: /PDB/Fuse_RTM -> /TSSI/GLV
- F5 pad 2: 12V -> /12V
- F6 pad 1: /PDB/Back_Car_12V -> Net-(J4-Pin_1)
- F6 pad 2: 12V -> /12V
- J12 pad 1: /PDB/Fuse_EXP1_12V -> /CCM Helper/CCM3v3
- J12 pad 2: GND -> /CCM Helper/RTDB
- J13 pad 1: /PDB/Fuse_EXP3_12V -> /CCM Helper/12V
- J13 pad 2: GND -> /CCM Helper/Brakelight
- J17 pad 1: 12V -> /CCM Helper/12V
- J17 pad 2: GND -> /CCM Helper/Speaker LPF'd
- J17 pad 3: 12V -> /CCM Helper/CCMGND
- J17 pad 4: Throttle_Sensor_Vout1 -> /CCM Helper/CCMGND
- J18 pad 1: 5V -> Net-(J18-VBUS)
- J18 pad 2: GND -> unconnected-(J18-D--Pad2)
- J18 pad 3: Wheel_Sensor_Vout1 -> unconnected-(J18-D+-Pad3)
- J18 pad 4: unconnected-(J18-Pin_4-Pad4) -> GND
- J8 pad 1: 5V -> +5V
- J8 pad 2: GND -> /BSPD/C_IN
- J8 pad 3: Linear_Pot1 -> unconnected-(J8-Pin_3-Pad3)
- J8 pad 4: unconnected-(J8-Pin_4-Pad4) -> GND
- J9 pad 1: 5V -> /TSSI/GLV
- J9 pad 2: GND -> /TSSI/GLV
- J9 pad 3: Linear_Pot2 -> /TSSI/GREEN_LED
- J9 pad 4: unconnected-(J9-Pin_4-Pad4) -> /TSSI/RED_LED
- R48 pad 1: /PDB/FB -> /CCM Helper/APPS2 IN
- R48 pad 2: GND -> /CCM Helper/APPS2 OUT
- R49 pad 1: Throttle_Sensor_Vout1 -> /CCM Helper/APPS1 IN
- R49 pad 2: GND -> /CCM Helper/APPS1 OUT
- R50 pad 1: Throttle_Sensor_Vout2 -> /CCM Helper/BPS1 IN
- R50 pad 2: GND -> /BSPD/B_IN
- SW2 pad 1: /LATCH/IMD_FAULT -> /IMD Fault
- U10 pad 1: /PDB/FB -> Net-(J18-VBUS)
- U10 pad 2: /PDB/BUCK_IN -> Net-(U10-TRIM)
- U10 pad 3: /PDB/BUCK_IN -> GND
- U10 pad 4: GND -> 12V_OUT
- U10 pad 5: /PDB/SW -> GND
Routing:
- net +12V: track 0.00 -> 353.7 mm
- net (no net): track 0.00 -> 108.2 mm
- net BSPD_FAULT: track 0.00 -> 96.8 mm
- net C_IN: track 0.00 -> 79.7 mm
- net OPEN_CIRCUIT: track 0.00 -> 67.1 mm
- net BRAKE: track 0.00 -> 65.8 mm
- net PEDAL_ERROR: track 0.00 -> 52.5 mm
- net CURRENT: track 0.00 -> 52.3 mm
- net BRAKE_ERROR: track 0.00 -> 49.0 mm
- net SHORT_CIRCUIT: track 0.00 -> 47.7 mm
- net BOTH_ON: track 0.00 -> 43.3 mm
- net PEDAL_SHORT: track 0.00 -> 42.5 mm
- net BRAKE_SHORT: track 0.00 -> 40.3 mm
- net PEDAL_THRESHOLD: track 0.00 -> 39.0 mm
- net BRAKE_APPLIED: track 0.00 -> 32.7 mm
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Other:
- board outline added: 90 x 70 mm
- board text added: "AND"
- board text added: "BRAKE"
- board text added: "BSPD 2026.3 Designed: Albert, Esmeralda Reviewed: Lucas, Gabriel"
- board text added: "LED1: Brake LED2: Current LED3: Simultaneous"
- board text added: "OC"
- board text added: "OR"
- board text added: "PEDAL"
- board text added: "SC"
- board text added: "Schmitt"

Commit message: hopefully this lets avadi pull
Parts:
- removed the C1 at (150.0, 272.7)
- removed the C1 at (46.2, 241.8)
- removed the C10 at (71.4, 286.3)
- removed the C10 at (154.1, 272.7)
- removed the C2 at (150.0, 275.2)
- removed the C2 at (66.9, 242.3)
- removed the C3 at (150.0, 277.7)
- removed the C3 at (47.2, 257.8)
- removed the C4 at (150.0, 280.2)
- removed the C4 at (66.4, 265.8)
- removed the C5 at (46.4, 274.8)
- removed the C5 at (150.0, 282.7)
- removed the C6 at (87.7, 265.0)
- removed the C6 at (150.0, 285.2)
- removed the C7 at (72.4, 271.8)
- removed the C7 at (150.0, 287.7)
- removed the C8 at (34.2, 289.3)
- removed the C8 at (150.0, 290.2)
- removed the C9 at (150.0, 292.7)
- removed the C9 at (34.2, 295.1)
- removed the D1 at (69.2, 266.6)
- removed the D1 at (177.7, 272.7)
- removed the D2 at (177.7, 275.3)
- removed the D2 at (36.7, 289.3)
- removed the H1 at (130.6, 275.2)
- removed the H1 at (14.2, 235.3)
- removed the H2 at (94.2, 235.3)
- removed the H2 at (130.6, 282.7)
- removed the H3 at (130.6, 290.3)
- removed the H3 at (14.2, 295.3)
- removed the H4 at (130.6, 297.8)
- removed the H4 at (94.2, 295.3)
- removed the J1 at (94.6, 269.8)
- removed the J1 at (238.9, 104.6)
- removed the J2 at (246.4, 104.6)
- removed the J2 at (49.0, 290.3)
- removed the Q1 at (75.9, 249.3)
- removed the Q1 at (137.8, 328.1)
- removed the R1 at (29.2, 241.8)
- removed the R1 at (154.1, 275.2)
- removed the R10 at (21.2, 273.8)
- removed the R10 at (158.1, 275.2)
- removed the R11 at (31.0, 258.0)
- removed the R11 at (158.1, 277.7)
- removed the R12 at (158.1, 280.2)
- removed the R12 at (46.7, 276.8)
- removed the R13 at (158.1, 282.7)
- removed the R13 at (47.4, 260.3)
- removed the R14 at (158.1, 285.2)
- removed the R14 at (72.4, 265.8)
- removed the R15 at (158.1, 287.7)
- removed the R15 at (72.4, 268.3)
- removed the R16 at (158.1, 290.2)
- removed the R16 at (20.7, 286.8)
- removed the R17 at (20.5, 281.8)
- removed the R17 at (158.1, 292.7)
- removed the R18 at (162.1, 272.7)
- removed the R18 at (38.9, 295.1)
- removed the R19 at (36.5, 295.1)
- removed the R19 at (162.1, 275.2)
- removed the R2 at (21.0, 248.3)
- removed the R2 at (154.1, 277.7)
- removed the R20 at (67.8, 286.3)
- removed the R20 at (162.1, 277.7)
- removed the R21 at (162.1, 280.2)
- removed the R21 at (67.7, 283.8)
- removed the R22 at (162.1, 282.7)
- removed the R22 at (49.1, 271.7)
- removed the R23 at (162.1, 285.2)
- removed the R23 at (67.8, 273.3)
- removed the R24 at (66.8, 279.0)
- removed the R24 at (162.1, 287.7)
- removed the R3 at (154.1, 280.2)
- removed the R3 at (21.0, 243.3)
- removed the R4 at (154.1, 282.7)
- removed the R4 at (47.5, 244.3)
- removed the R5 at (154.1, 285.2)
- removed the R5 at (74.8, 244.6)
- removed the R6 at (154.1, 287.7)
- removed the R6 at (21.2, 256.3)
- removed the R7 at (21.2, 261.3)
- removed the R7 at (154.1, 290.2)
- removed the R8 at (154.1, 292.7)
- removed the R8 at (21.0, 268.8)
- removed the R9 at (158.1, 272.7)
- removed the R9 at (30.4, 274.3)
- removed the R_Bypass1 at (162.1, 290.2)
- removed the R_Bypass1 at (77.7, 287.9)
- removed the R_Bypass2 at (83.2, 287.9)
- removed the R_Bypass2 at (162.1, 292.7)
- removed the TP1 at (136.7, 273.7)
- removed the TP1 at (30.2, 237.3)
- removed the TP10 at (141.2, 287.3)
- removed the TP10 at (25.7, 258.8)
- removed the TP11 at (141.2, 291.9)
- removed the TP11 at (36.2, 270.8)
- removed the TP12 at (48.7, 263.3)
- removed the TP12 at (141.2, 296.4)
- removed the TP13 at (80.1, 259.6)
- removed the TP13 at (145.8, 273.7)
- removed the TP14 at (30.8, 294.3)
- removed the TP14 at (145.8, 278.2)
- removed the TP15 at (25.2, 284.3)
- removed the TP15 at (145.8, 282.8)
- removed the TP16 at (145.8, 287.3)
- removed the TP16 at (52.7, 284.2)
- removed the TP17 at (47.2, 284.3)
- removed the TP17 at (145.8, 291.9)
- removed the TP2 at (25.2, 245.8)
- removed the TP2 at (136.7, 278.2)
- removed the TP3 at (47.2, 248.8)
- removed the TP3 at (136.7, 282.8)
- removed the TP4 at (136.7, 287.3)
- removed the TP4 at (64.7, 238.3)
- removed the TP5 at (69.9, 249.8)
- removed the TP5 at (136.7, 291.9)
- removed the TP6 at (60.7, 238.3)
- removed the TP6 at (136.7, 296.4)
- removed the TP7 at (141.2, 273.7)
- removed the TP7 at (67.2, 246.8)
- removed the TP8 at (25.2, 271.3)
- removed the TP8 at (141.2, 278.2)
- removed the TP9 at (141.2, 282.8)
- removed the TP9 at (29.7, 261.3)
- removed the U1 at (34.9, 242.0)
- removed the U1 at (150.1, 296.1)
- removed U10: OKX-T/5-D12N-C, footprints:12v5vDCDC
- removed the U2 at (161.8, 296.1)
- removed the U2 at (55.6, 242.2)
- removed the U3 at (34.9, 258.0)
- removed the U3 at (167.3, 291.6)
- removed the U4 at (150.1, 315.6)
- removed the U4 at (34.9, 274.5)
- removed the U5 at (55.4, 265.7)
- removed the U5 at (161.8, 315.6)
- removed the U6 at (77.1, 265.8)
- removed the U6 at (173.5, 296.1)
- removed the VR1 at (12.2, 243.3)
- removed the VR1 at (142.5, 300.6)
- removed the VR2 at (142.5, 307.0)
- removed the VR2 at (12.2, 256.2)
- removed the VR3 at (142.5, 313.4)
- removed the VR3 at (12.2, 268.8)
- removed the VR4 at (142.5, 319.8)
- removed the VR4 at (12.2, 281.8)
- added C1: 10u, Capacitor_SMD:C_0603_1608Metric, F.Cu at (231.8, 42.3)
- added C10: 0.1u, Capacitor_SMD:C_0603_1608Metric, F.Cu at (235.8, 42.3)
- added C2: 1n, Capacitor_SMD:C_0603_1608Metric, F.Cu at (231.8, 44.8)
- added C3: 1n, Capacitor_SMD:C_0603_1608Metric, F.Cu at (231.8, 47.3)
- added C32: 330uF, Capacitor_SMD:C_2220_5750Metric_Pad1.97x5.40mm_HandSolder, F.Cu at (448.0, 101.7)
- added C4: 3.3u, Capacitor_SMD:C_0603_1608Metric, F.Cu at (231.8, 49.8)
- added C5: 0.1u, Capacitor_SMD:C_0603_1608Metric, F.Cu at (231.8, 52.3)
- added C6: 0.1u, Capacitor_SMD:C_0603_1608Metric, F.Cu at (231.8, 54.8)
- added C7: 0.1u, Capacitor_SMD:C_0603_1608Metric, F.Cu at (231.8, 57.3)
- added C8: 0.1u, Capacitor_SMD:C_0603_1608Metric, F.Cu at (231.8, 59.9)
- added C9: 0.1u, Capacitor_SMD:C_0603_1608Metric, F.Cu at (231.8, 62.4)
- added D1: D, Diode_SMD:D_0603_1608Metric, F.Cu at (271.8, 84.4)
- added D2: D, Diode_SMD:D_0603_1608Metric, F.Cu at (271.8, 87.0)
- added F10: ~, 0footprints:FUSE_3522-2, F.Cu at (449.2, 148.1)
- added F7: ~, 0footprints:FUSE_3522-2, F.Cu at (510.7, 160.1)
- added F8: ~, 0footprints:FUSE_3522-2, F.Cu at (493.3, 101.1)
- added F9: ~, 0footprints:FUSE_3522-2, F.Cu at (449.2, 142.1)
- added H1: MH, MountingHole:MountingHole_3mm, F.Cu at (212.4, 44.8)
- added H2: MH, MountingHole:MountingHole_3mm, F.Cu at (212.4, 52.4)
- added H3: MH, MountingHole:MountingHole_3mm, F.Cu at (212.4, 59.9)
- added H4: MH, MountingHole:MountingHole_3mm, F.Cu at (212.4, 67.5)
- added J1: ESTOP/SDC switch, 0footprints:Molex_Mini-Fit_Jr_5566-02A_2x01_P4.20mm_Vertical, F.Cu at (165.4, 21.6)
- added J10: Dash, footprints:Molex_Mini-Fit_Jr_5566-06A_2x03_P4.20mm_Vertical, F.Cu at (193.3, 19.8)
- added J11: BBC, footprints:12pSTminifit, F.Cu at (83.3, 253.7)
- added J14: Brakelight, 0footprints:Molex_Mini-Fit_Jr_5566-02A_2x01_P4.20mm_Vertical, F.Cu at (89.9, 74.6)
- added J15: SHOCK/WHEEL SNSR, footprints:12pSTminifit, F.Cu at (53.8, 74.4)
- added J19: 39306207, footprints:20pSTminfit, F.Cu at (88.5, 125.8)
- added J2: SDC OUT, 0footprints:Molex_Mini-Fit_Jr_5566-02A_2x01_P4.20mm_Vertical, F.Cu at (210.8, 264.8)
- added K1: G6B-2214P-US DC12, footprints:DPSTrelay, F.Cu at (71.2, 248.7)
- added K2: G6B-2214P-US DC12, footprints:DPSTrelay, F.Cu at (83.7, 248.7)
- added K3: G6B-2214P-US DC12, footprints:DPSTrelay, F.Cu at (96.3, 248.7)
- added Q1: IRLIZ44N NMOS, Package_TO_SOT_THT:TO-220F-3_Horizontal_TabDown, F.Cu at (260.8, 60.9)
- added Q2: IRLIZ44N NMOS, Package_TO_SOT_THT:TO-220F-3_Horizontal_TabDown, F.Cu at (315.1, 224.6)
- added Q3: IRLIZ44N NMOS, Package_TO_SOT_THT:TO-220F-3_Horizontal_TabDown, F.Cu at (326.9, 224.6)
- added Q7: PMOS IRF9540, Package_TO_SOT_THT:TO-220-3_Vertical, F.Cu at (102.0, 244.9)
- added R1: 500k, Resistor_SMD:R_0603_1608Metric, F.Cu at (235.8, 44.8)
- added R10: 10K, Resistor_SMD:R_0603_1608Metric, F.Cu at (239.9, 44.8)
- added R11: 10K, Resistor_SMD:R_0603_1608Metric, F.Cu at (239.9, 47.3)
- added R12: 10K, Resistor_SMD:R_0603_1608Metric, F.Cu at (239.9, 49.8)
- added R13: 10K, Resistor_SMD:R_0603_1608Metric, F.Cu at (239.9, 52.3)
- added R14: 10K, Resistor_SMD:R_0603_1608Metric, F.Cu at (239.9, 54.8)
- added R15: 10K, Resistor_SMD:R_0603_1608Metric, F.Cu at (239.9, 57.3)
- added R16: 10k, Resistor_SMD:R_0603_1608Metric, F.Cu at (239.9, 59.9)
- added R17: 20k, Resistor_SMD:R_0603_1608Metric, F.Cu at (239.9, 62.4)
- added R18: 20k, Resistor_SMD:R_0603_1608Metric, F.Cu at (243.9, 42.3)
- added R19: 20k, Resistor_SMD:R_0603_1608Metric, F.Cu at (243.9, 44.8)
- added R2: 500k, Resistor_SMD:R_0603_1608Metric, F.Cu at (235.8, 47.3)
- added R20: 20k, Resistor_SMD:R_0603_1608Metric, F.Cu at (243.9, 47.3)
- added R21: 120k, Resistor_SMD:R_0603_1608Metric, F.Cu at (243.9, 49.8)
- added R22: 1k, Resistor_SMD:R_0603_1608Metric, F.Cu at (243.9, 52.3)
- added R23: 20k, Resistor_SMD:R_0603_1608Metric, F.Cu at (243.9, 54.8)
- added R24: 20k, Resistor_SMD:R_0603_1608Metric, F.Cu at (243.9, 57.3)
- added R25: 1k, Resistor_SMD:R_0805_2012Metric, F.Cu at (336.3, 236.9)
- added R3: 1k, Resistor_SMD:R_0603_1608Metric, F.Cu at (235.8, 49.8)
- added R4: 10k, Resistor_SMD:R_0603_1608Metric, F.Cu at (235.8, 52.3)
- added R5: 1k, Resistor_SMD:R_0603_1608Metric, F.Cu at (235.8, 54.8)
- added R59: 1k, Resistor_SMD:R_0805_2012Metric, F.Cu at (89.8, 100.7)
- added R6: 10k, Resistor_SMD:R_0603_1608Metric, F.Cu at (235.8, 57.3)
- added R7: 10k, Resistor_SMD:R_0603_1608Metric, F.Cu at (235.8, 59.9)
- added R8: 10K, Resistor_SMD:R_0603_1608Metric, F.Cu at (235.8, 62.4)
- added R9: 10K, Resistor_SMD:R_0603_1608Metric, F.Cu at (239.9, 42.3)
- added R_Bypass1: 0, Resistor_SMD:R_0603_1608Metric, F.Cu at (243.9, 59.9)
- added R_Bypass2: 0, Resistor_SMD:R_0603_1608Metric, F.Cu at (243.9, 62.4)
- added TP1: BRAKE, TestPoint:TestPoint_Pad_D2.5mm, F.Cu at (218.5, 43.3)
- added TP10: B_SHORT, TestPoint:TestPoint_Pad_D2.5mm, F.Cu at (223.0, 57.0)
- added TP11: B_OPEN, TestPoint:TestPoint_Pad_D2.5mm, F.Cu at (223.0, 61.5)
- added TP12: P_SHORT, TestPoint:TestPoint_Pad_D2.5mm, F.Cu at (223.0, 66.1)
- added TP13: P_OPEN, TestPoint:TestPoint_Pad_D2.5mm, F.Cu at (227.6, 43.3)
- added TP14: B_ERROR, TestPoint:TestPoint_Pad_D2.5mm, F.Cu at (227.6, 47.9)
- added TP15: P_ERROR, TestPoint:TestPoint_Pad_D2.5mm, F.Cu at (227.6, 52.4)
- added TP16: FAULT_SENSED, TestPoint:TestPoint_Pad_D2.5mm, F.Cu at (227.6, 57.0)
- added TP17: BSPD_FAULT, TestPoint:TestPoint_Pad_D2.5mm, F.Cu at (227.6, 61.5)
- added TP2: PEDAL, TestPoint:TestPoint_Pad_D2.5mm, F.Cu at (218.5, 47.9)
- added TP3: SC, TestPoint:TestPoint_Pad_D2.5mm, F.Cu at (218.5, 52.4)
- added TP4: OC, TestPoint:TestPoint_Pad_D2.5mm, F.Cu at (218.5, 57.0)
- added TP5: BRAKE_TH, TestPoint:TestPoint_Pad_D2.5mm, F.Cu at (218.5, 61.5)
- added TP6: PEDAL_TH, TestPoint:TestPoint_Pad_D2.5mm, F.Cu at (218.5, 66.1)
- added TP7: B_APPLIED, TestPoint:TestPoint_Pad_D2.5mm, F.Cu at (223.0, 43.3)
- added TP8: P_APPLIED, TestPoint:TestPoint_Pad_D2.5mm, F.Cu at (223.0, 47.9)
- added TP9: BOTH_ON, TestPoint:TestPoint_Pad_D2.5mm, F.Cu at (223.0, 52.4)
- added U1: 40106 Inverter, Package_DIP:DIP-14_W7.62mm_Socket, F.Cu at (231.9, 65.7)
- added U2: 4081 AND Gate, Package_DIP:DIP-14_W7.62mm_Socket, F.Cu at (243.6, 65.7)
- added U3: LT1084-5.0, Package_TO_SOT_THT:TO-220-3_Horizontal_TabDown, F.Cu at (284.8, 63.1)
- added U4: LM393, Package_DIP:DIP-8_W7.62mm_Socket, F.Cu at (231.9, 85.2)
- added U5: LM393, Package_DIP:DIP-8_W7.62mm_Socket, F.Cu at (243.6, 85.2)
- added U6: 4071 4 Channel 2 Input OR gate, Package_DIP:DIP-14_W7.62mm_Socket, F.Cu at (255.3, 65.7)
- added U9: OKX-T/5-D12N-C, footprints:12v5vDCDC, F.Cu at (449.6, 116.7)
- added VR1: 3296Y-11-103LF, Potentiometer_THT:Potentiometer_Bourns_3296Y_Vertical, F.Cu at (224.3, 70.2)
- added VR2: 3296Y-11-103LF, Potentiometer_THT:Potentiometer_Bourns_3296Y_Vertical, F.Cu at (224.3, 76.6)
- added VR3: 3296Y-11-103LF, Potentiometer_THT:Potentiometer_Bourns_3296Y_Vertical, F.Cu at (224.3, 83.0)
- added VR4: 3296Y-11-103LF, Potentiometer_THT:Potentiometer_Bourns_3296Y_Vertical, F.Cu at (224.3, 89.4)
- C16: value 1u -> 330uF; footprint Capacitor_SMD:C_0805_2012Metric -> Capacitor_SMD:C_2220_5750Metric_Pad1.97x5.40mm_HandSolder
- C17: value 1u -> 22uF
- C18: value 330uF -> 1u; footprint Capacitor_SMD:C_2220_5750Metric_Pad1.97x5.40mm_HandSolder -> Capacitor_SMD:C_0805_2012Metric
- C19: value 22uF -> 1u
- C20: value 10n -> 1u
- C21: value 22uF -> 330uF; footprint Capacitor_SMD:C_0805_2012Metric -> Capacitor_SMD:C_2220_5750Metric_Pad1.97x5.40mm_HandSolder
- C22, C23: value 100n -> 22uF
- C24: value 100n -> 10u
- C25: value 100n -> 330uF; footprint Capacitor_SMD:C_0805_2012Metric -> Capacitor_SMD:C_2220_5750Metric_Pad1.97x5.40mm_HandSolder
- C26: value 330uF -> 10n; footprint Capacitor_SMD:C_2220_5750Metric_Pad1.97x5.40mm_HandSolder -> Capacitor_SMD:C_0805_2012Metric
- C27: value 330uF -> 22uF; footprint Capacitor_SMD:C_2220_5750Metric_Pad1.97x5.40mm_HandSolder -> Capacitor_SMD:C_0805_2012Metric
- C28, C29: value 22uF -> 100n
- C30: value 10u -> 100n
- C31: value 330uF -> 100n; footprint Capacitor_SMD:C_2220_5750Metric_Pad1.97x5.40mm_HandSolder -> Capacitor_SMD:C_0805_2012Metric
- J12: value RTD B -> 614004135023; footprint 0footprints:Molex_Mini-Fit_Jr_5566-02A_2x01_P4.20mm_Vertical -> footprints:614004135023
- J13: value Brakelight -> RTD B
- J17: value Conn_01x04_Pin -> Pedal snsrs; footprint footprints:AmpBoard -> footprints:12pSTminifit
- J18: value 614004135023 -> AMP; footprint footprints:614004135023 -> footprints:AmpBoard
- J3: value SDC OUT -> ACCU; footprint 0footprints:Molex_Mini-Fit_Jr_5566-02A_2x01_P4.20mm_Vertical -> 0footprints:Molex_Mini-Fit_Jr_5566-04A_2x02_P4.20mm_Vertical
- J4: value ACCU -> 12v EXP; footprint 0footprints:Molex_Mini-Fit_Jr_5566-04A_2x02_P4.20mm_Vertical -> 0footprints:Molex_Mini-Fit_Jr_5566-02A_2x01_P4.20mm_Vertical
- J5: value BSPD -> PWR IN; footprint 0footprints:Molex_Mini-Fit_Jr_5566-06A_2x03_P4.20mm_Vertical -> 0footprints:Molex_Mini-Fit_Jr_5566-02A_2x01_P4.20mm_Vertical
- J6: value LATCH -> 24v EXP; footprint 0footprints:Molex_Mini-Fit_Jr_5566-08A_2x04_P4.20mm_Vertical -> 0footprints:Molex_Mini-Fit_Jr_5566-02A_2x01_P4.20mm_Vertical
- J7: value ACCU -> 5v EXP; footprint 0footprints:Molex_Mini-Fit_Jr_5566-04A_2x02_P4.20mm_Vertical -> 0footprints:Molex_Mini-Fit_Jr_5566-02A_2x01_P4.20mm_Vertical
- LED1, LED2, LED3: footprint SMALL_LED:LEDC2012X105N -> LED_SMD:LED_0805_2012Metric_Pad1.15x1.40mm_HandSolder
- Q4: value PMOS IRF9540 -> IRLIZ44N NMOS; footprint Package_TO_SOT_THT:TO-220-3_Vertical -> Package_TO_SOT_THT:TO-220F-3_Horizontal_TabDown
- R26: value 13k -> 1k
- R27: value 4k -> 13k
- R28: value 22k -> 4k
- R31: value 220k -> 22k
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Connections:
- C16 pad 1: /CCM Helper/BPS1 IN -> /5V
- C16 pad 2: /CCM Helper/CCMGND -> GND
- C17 pad 1: /CCM Helper/BPS2 IN -> /5V
- C17 pad 2: /CCM Helper/CCMGND -> GND
- C18 pad 1: Net-(FL1-VOUT(+)_) -> /CCM Helper/BPS1 IN
- C18 pad 2: GND -> /CCM Helper/CCMGND
- C19 pad 1: Net-(FL1-VOUT(+)_) -> /CCM Helper/BPS2 IN
- C19 pad 2: GND -> /CCM Helper/CCMGND
- C20 pad 1: /CCM Helper/Speaker IN -> Net-(FL1-CASE)
- C20 pad 2: /CCM Helper/CCMGND -> GND
- C21 pad 1: 12V_OUT -> Net-(FL1-VOUT(+)_)
- C22 pad 1: /CCM Helper/Wheel/Shock1 IN -> Net-(FL1-VOUT(+)_)
- C22 pad 2: /CCM Helper/CCMGND -> GND
- C23 pad 1: /CCM Helper/Wheel/Shock2 IN -> /24V
- C23 pad 2: /CCM Helper/CCMGND -> GND
- C24 pad 1: /CCM Helper/Wheel/Shock3 IN -> /24V
- C24 pad 2: /CCM Helper/CCMGND -> GND
- C25 pad 1: /CCM Helper/Wheel/Shock4 IN -> /24V
- C25 pad 2: /CCM Helper/CCMGND -> GND
- C26 pad 1: 12V_OUT -> /CCM Helper/Speaker IN
- C26 pad 2: GND -> /CCM Helper/CCMGND
- C27 pad 1: Net-(J18-VBUS) -> /24V
- C28 pad 1: Net-(J18-VBUS) -> /CCM Helper/Wheel/Shock1 IN
- C28 pad 2: GND -> /CCM Helper/CCMGND
- C29 pad 1: 12V_OUT -> /CCM Helper/Wheel/Shock2 IN
- C29 pad 2: GND -> /CCM Helper/CCMGND
- C30 pad 1: 12V_OUT -> /CCM Helper/Wheel/Shock3 IN
- C30 pad 2: GND -> /CCM Helper/CCMGND
- C31 pad 1: 12V_OUT -> /CCM Helper/Wheel/Shock4 IN
- C31 pad 2: GND -> /CCM Helper/CCMGND
- F2 pad 1: /12V_2 -> +12V
- F6 pad 1: Net-(J4-Pin_1) -> Net-(J3-Pin_1)
- FL1 pad 2: 24V_IN -> /12V
- FL1 pad 3: unconnected-(FL1-CASE-Pad3) -> Net-(FL1-CASE)
- J12 pad 1: /CCM Helper/CCM3v3 -> /5V
- J12 pad 2: /CCM Helper/RTDB -> unconnected-(J12-D--Pad2)
- J13 pad 1: /CCM Helper/12V -> /CCM Helper/CCM3v3
- J13 pad 2: /CCM Helper/Brakelight -> /CCM Helper/RTDB
- J17 pad 1: /CCM Helper/12V -> /CCM Helper/CCM3v3
- J17 pad 2: /CCM Helper/Speaker LPF'd -> /CCM Helper/CCMGND
- J17 pad 3: /CCM Helper/CCMGND -> /CCM Helper/APPS1 IN
- J17 pad 4: /CCM Helper/CCMGND -> /CCM Helper/CCM3v3
- J18 pad 1: Net-(J18-VBUS) -> /CCM Helper/12V
- J18 pad 2: unconnected-(J18-D--Pad2) -> /CCM Helper/Speaker LPF'd
- J18 pad 3: unconnected-(J18-D+-Pad3) -> /CCM Helper/CCMGND
- J18 pad 4: GND -> /CCM Helper/CCMGND
- J3 pad 1: /24V -> Net-(J3-Pin_1)
- J5 pad 1: unconnected-(J5-Pin_1-Pad1) -> Net-(J5-Pin_1)
- J5 pad 2: unconnected-(J5-Pin_2-Pad2) -> GND
- J6 pad 1: unconnected-(J6-Pin_1-Pad1) -> Net-(J6-Pin_1)
- J6 pad 2: unconnected-(J6-Pin_2-Pad2) -> GND
- J7 pad 1: unconnected-(J7-Pin_1-Pad1) -> Net-(J7-Pin_1)
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Routing:
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Other:
- board outline removed
- board text removed: "AND"
- board text removed: "BRAKE"
- board text removed: "BSPD 2026.3 Designed: Albert, Esmeralda Reviewed: Lucas, Gabriel"
- board text removed: "LED1: Brake LED2: Current LED3: Simultaneous"
- board text removed: "OC"
- board text removed: "OR"
- board text removed: "PEDAL"
- board text removed: "SC"
- board text removed: "Schmitt"

Commit message: rough layout done
Parts:
- removed D13: SB560-3G, Diode_THT:D_DO-201_P15.24mm_Horizontal
- removed H10, H11, H12, H9: MountingHole, MountingHole:MountingHole_3.2mm_M3
- removed J17: Pedal snsrs, footprints:12pSTminifit
- removed R38, R43, R48: 0, Resistor_THT:R_Axial_DIN0207_L6.3mm_D2.5mm_P10.16mm_Horizontal
- removed R39, R44: 470, Resistor_THT:R_Axial_DIN0207_L6.3mm_D2.5mm_P10.16mm_Horizontal
- removed T1: Test555, Connector_PinHeader_1.00mm:PinHeader_1x01_P1.00mm_Vertical
- removed TP1: BRAKE, TestPoint:TestPoint_Pad_D2.5mm
- removed TP10: B_SHORT, TestPoint:TestPoint_Pad_D2.5mm
- removed TP11: B_OPEN, TestPoint:TestPoint_Pad_D2.5mm
- removed TP12: P_SHORT, TestPoint:TestPoint_Pad_D2.5mm
- removed TP13: P_OPEN, TestPoint:TestPoint_Pad_D2.5mm
- removed TP14: B_ERROR, TestPoint:TestPoint_Pad_D2.5mm
- removed TP15: P_ERROR, TestPoint:TestPoint_Pad_D2.5mm
- removed TP16: FAULT_SENSED, TestPoint:TestPoint_Pad_D2.5mm
- removed TP17: BSPD_FAULT, TestPoint:TestPoint_Pad_D2.5mm
- removed TP2: PEDAL, TestPoint:TestPoint_Pad_D2.5mm
- removed TP3: SC, TestPoint:TestPoint_Pad_D2.5mm
- removed TP4: OC, TestPoint:TestPoint_Pad_D2.5mm
- removed TP5: BRAKE_TH, TestPoint:TestPoint_Pad_D2.5mm
- removed TP6: PEDAL_TH, TestPoint:TestPoint_Pad_D2.5mm
- removed TP7: B_APPLIED, TestPoint:TestPoint_Pad_D2.5mm
- removed TP8: P_APPLIED, TestPoint:TestPoint_Pad_D2.5mm
- removed TP9: BOTH_ON, TestPoint:TestPoint_Pad_D2.5mm
- added F11: ~, 0footprints:FUSE_3522-2, F.Cu at (260.8, 123.1)
- added F12: ~, 0footprints:FUSE_3522-2, F.Cu at (277.1, 154.7)
- added J16: footwell, footprints:14pSTminifit, F.Cu at (112.5, 130.9)
- C1, C10, C11, C12, C13, C14, C15, C16, C17, C18, C19, C2, C20, C21, C22, C23, C24, C25, C27, C28, C29, C3, C30, C31, C32, C5, C6, C7, C8, C9, D1, D2, Q2, Q3, R1, R10, R11, R12, R13, R14, R15, R17, R18, R19, R2, R20, R21, R23, R24, R3, R31, R32, R4, R49, R5, R50, R51, R52, R53, R55, R56, R57, R58, R59, R6, R7, R8, R9: moved to B.Cu
- D10: value SB560-3G -> D; footprint Diode_THT:D_DO-201_P15.24mm_Horizontal -> Diode_SMD:D_0603_1608Metric
- D11, D6, D8: value SB560-3G -> D; footprint Diode_THT:D_DO-201_P15.24mm_Horizontal -> Diode_SMD:D_0603_1608Metric; moved to B.Cu
- Q5, Q6, Q7: footprint Package_TO_SOT_THT:TO-220-3_Vertical -> Package_TO_SOT_THT:TO-220F-3_Horizontal_TabDown; moved to B.Cu
- R30: value 22k -> 10k
- R34: value 470 -> 22k; footprint Resistor_THT:R_Axial_DIN0207_L6.3mm_D2.5mm_P10.16mm_Horizontal -> Resistor_SMD:R_0805_2012Metric; moved to B.Cu
- R35, R36, R37, R40, R41, R45, R46, R47: footprint Resistor_THT:R_Axial_DIN0207_L6.3mm_D2.5mm_P10.16mm_Horizontal -> Resistor_SMD:R_0805_2012Metric_Pad1.20x1.40mm_HandSolder
- R42: footprint Resistor_THT:R_Axial_DIN0207_L6.3mm_D2.5mm_P10.16mm_Horizontal -> Resistor_SMD:R_0805_2012Metric_Pad1.20x1.40mm_HandSolder; moved to B.Cu
- moved H1 430.9 mm to (642.9, 24.7)
- moved H2 430.9 mm to (642.9, 32.2)
- moved H3 430.9 mm to (642.9, 39.8)
- moved H4 430.9 mm to (642.9, 47.3)
- moved F1 383.5 mm to (678.4, 62.7)
- moved J5 373.2 mm to (127.4, 132.3), turned to 90 degrees
- moved F8 360.9 mm to (134.6, 140.6), turned to 180 degrees
- moved J6 350.9 mm to (127.4, 157.6), turned to 90 degrees
- moved R28 333.3 mm to (9.59, 199.0)
- moved R27 333.1 mm to (6.14, 199.0)
- moved R25 315.9 mm to (23.4, 194.0)
- moved F9 314.7 mm to (134.6, 149.0), turned to 180 degrees
- moved D3 313.1 mm to (15.2, 198.9), turned to 180 degrees
- moved R26 312.5 mm to (27.2, 194.0)
- moved F2 287.4 mm to (402.9, 126.0)
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Connections:
- C23 pad 1: /24V -> /12V
- C24 pad 1: /24V -> /12V
- C25 pad 1: /24V -> /12V
- C27 pad 1: /24V -> Net-(PS1-SENSE+)
- C32 pad 1: /24V -> Net-(PS1-SENSE+)
- D1 pad 1: GND -> /LATCH/bspd_reset
- D1 pad 2: +12V -> /BSPD/BSPD_FAULT
- D10 pad 1: /LATCH/imd_reset -> /LATCH/bms_reset
- D10 pad 2: GND -> /BMS FAULT
- D8 pad 1: /LATCH/bspd_reset -> /LATCH/imd_reset
- D8 pad 2: /BSPD/BSPD_FAULT -> GND
- FL1 pad 2: /12V -> /24V
- J12 pad 1: /5V -> Net-(J12-VBUS)
- J15 pad 10: /CCM Helper/CCMGND -> /CCM Helper/Wheel/Shock2 IN
- J15 pad 12: /CCM Helper/CCMGND -> /CCM Helper/Wheel/Shock4 IN
- J15 pad 2: /CCM Helper/Wheel/Shock4 IN -> /CCM Helper/5V
- J15 pad 4: /CCM Helper/5V -> /CCM Helper/CCMGND
- J15 pad 5: /CCM Helper/5V -> /CCM Helper/CCMGND
- J15 pad 6: /CCM Helper/5V -> /CCM Helper/CCMGND
- J15 pad 7: /CCM Helper/Wheel/Shock1 IN -> /CCM Helper/5V
- J15 pad 8: /CCM Helper/CCMGND -> /CCM Helper/5V
- J15 pad 9: /CCM Helper/Wheel/Shock2 IN -> /CCM Helper/Wheel/Shock1 IN
- J19 pad 1: GND -> /CCM Helper/TSSI BYP
- J19 pad 10: /CCM Helper/APPS2 OUT -> unconnected-(J19-Pad10)
- J19 pad 11: /CCM Helper/APPS1 OUT -> unconnected-(J19-Pad11)
- J19 pad 13: /CCM Helper/Speaker IN -> unconnected-(J19-Pad13)
- J19 pad 18: /CCM Helper/BPS2 OUT -> unconnected-(J19-Pad18)
- J19 pad 19: /BSPD/B_IN -> unconnected-(J19-Pad19)
- J19 pad 2: /CCM Helper/Brakelight -> /CCM Helper/CCM fdbk
- J19 pad 20: /CCM Helper/CCM3v3 -> /CCM Helper/Brakelight
- J19 pad 3: /CCM Helper/12V -> /CCM Helper/Speaker IN
- J19 pad 5: /CCM Helper/RTDB -> /BSPD/B_IN
- J19 pad 6: /CCM Helper/5V -> /CCM Helper/BPS2 OUT
- J19 pad 7: /CCM Helper/CCM fdbk -> /CCM Helper/CCM3v3
- J19 pad 8: /CCM Helper/TSSI BYP -> /CCM Helper/APPS1 OUT
- J19 pad 9: unconnected-(J19-Pad9) -> /CCM Helper/APPS2 OUT
- PS1 pad 12: /24V -> Net-(PS1-SENSE+)
- PS1 pad 7: /24V -> Net-(PS1-SENSE+)
- PS1 pad 8: /24V -> Net-(PS1-SENSE+)
- Q5 pad 2: Net-(Q5-D) -> /LATCH/BSPDfault_LED
- Q6 pad 2: Net-(Q6-D) -> /LATCH/IMDfault_LED
- Q7 pad 2: Net-(Q7-D) -> /LATCH/BMSfault_LED
- R34 pad 1: /LATCH/BSPDfault_LED -> Net-(D3-K)
- R34 pad 2: Net-(Q5-D) -> GND
- U9 pad 4: /24V -> /12V
Routing:
- net /BSPD/BOTH_ON: track 0.00 -> 58.7 mm, vias 0 -> 3
- net /BSPD/BRAKE: track 0.00 -> 53.8 mm, vias 0 -> 1
- net /BSPD/CURRENT: track 0.00 -> 47.8 mm, vias 0 -> 1
- net /BSPD/OPEN_CIRCUIT: track 0.00 -> 37.0 mm
- net +12V: track 0.00 -> 35.0 mm
- net /BSPD/PEDAL_ERROR: track 0.00 -> 28.7 mm
- net /BSPD/BRAKE_ERROR: track 0.00 -> 26.3 mm
- net /BSPD/SHORT_CIRCUIT: track 0.00 -> 24.0 mm, vias 0 -> 2
- net /BSPD/BRAKE_APPLIED: track 0.00 -> 23.3 mm, vias 0 -> 1
- net Net-(C4-Pad1): track 0.00 -> 22.4 mm, vias 0 -> 1
- net +5V: track 0.00 -> 21.0 mm
- net /BSPD/PEDAL_THRESHOLD: track 0.00 -> 18.2 mm
- net Net-(R6-Pad1): track 0.00 -> 17.6 mm, vias 0 -> 1
- net /BSPD/BRAKE_SHORT: track 0.00 -> 17.5 mm
- net /BSPD/PEDAL_APPLIED: track 0.00 -> 16.5 mm, vias 0 -> 1
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Other:
- board text added: "dont forget LDO caps!"
- board text added: "dont forget caps"
