File: SafetyBoard/SafetyBoard.kicad_sch (KiCad schematic)
At the start: 18 parts, among them J1 Estop, J2 TS ON SW, J3 SDC OUT, J4 ACCU, J5 12v EXP, J6 PWR IN, J7 24v EXP, J8 5v EXP

Commit message: Traces Check 2
Connections:
- net 12V: now also F7.2; no longer F7.1
- net at J5.1 (Pin_1): now also F7.1; no longer F7.2
Other:
- moved on the sheet: F7
Changed lines of the file:
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@@
 	(symbol
 		(lib_id "Device:Fuse")
-		(at 231.394 49.784 90)
+		(at 231.394 49.784 270)
 		(unit 1)
 		(exclude_from_sim no)
@@
 		(dnp no)
 		(property "Reference" "F7"
-			(at 231.394 47.498 90)
+			(at 231.394 52.07 90)
 			(effects
 				(font
@@
 		)
 		(property "Value" "5A MAX"
-			(at 231.394 51.562 90)
+			(at 231.394 48.006 90)
 			(effects
 				(font
@@
 		)
 		(property "Footprint" "0footprints:FUSE_3522-2"
-			(at 231.394 51.562 90)
+			(at 231.394 48.006 90)
 			(effects
 				(font
