File: TSSI/TSSI/TSSI.kicad_sch (KiCad schematic)
At the start: 26 parts, among them J1 Conn_02x02, J3 Conn_02x02, Q1 IRLZ34N, Q3 IRLZ34N, T555 Test555, U1 LM555xN, U3 IRLZ34N

Commit message: Changed a buncha stuff on other ppl's board. established new branch
Parts:
- removed CCM1: TestCCMCtrl, Connector_PinHeader_1.00mm:PinHeader_1x01_P1.00mm_Vertical, symbol Connector:Conn_01x01_Pin
- removed J1, J3: Conn_02x02, Connector_Molex:Molex_Mini-Fit_Jr_5566-04A2_2x02_P4.20mm_Vertical, symbol Connector_Generic:Conn_02x02_Counter_Clockwise
- removed Latch1: TestLatch, Connector_PinHeader_1.00mm:PinHeader_1x01_P1.00mm_Vertical, symbol Connector:Conn_01x01_Pin
- renumbered C1 to C11, C2 to C12, C3 to C13, D2 to D3, D3 to D4, D1 to D5, H1 to H5, H2 to H6, H3 to H7, H4 to H8, Q1 to Q2, R4 to R25, R5 to R26, R2 to R27, R1 to R28, R6 to R29, R7 to R30, R8 to R31, T555 to T1, U1 to U7, U3 to U8
Connections:
- net Latch_12V_Safe renamed Latch_Control
- no-connect marks 1 -> 0

Commit message: day 2 grind
Parts:
- added J9: TSSI, 0footprints:Molex_Mini-Fit_Jr_5566-04A_2x02_P4.20mm_Vertical, symbol Connector_Generic:Conn_02x02_Top_Bottom
- added R25: R_US, symbol Device:R_US
- renumbered R25 to R26, R26 to R27, R27 to R28, R28 to R29, R29 to R30, R30 to R31, R31 to R32, U7 to U8, U8 to U9
Connections:
- net GLV: now also J9.1 (Pin_1), J9.2 (Pin_2), R25.1; no longer Q2.GND
- net GND: now also Q2.GND
- net GREEN_LED: now also J9.3 (Pin_3)
- net RED_LED: now also J9.4 (Pin_4)
- net at D4.2 (A), Q2.OUT: now also R25.2
Other:
- moved on the sheet: Q2

Commit message: hopefully this lets avadi pull
Parts:
- removed Q2, Q3, U9: IRLZ34N, IRLZ34N:TO-220_2_, symbol IRLZ34N:IRLZ34N
- added Q2, Q3, Q4: IRLIZ44N NMOS, Package_TO_SOT_THT:TO-220F-3_Horizontal_TabDown, symbol Transistor_FET:IRLIZ44N
- added R26: 1k, Resistor_SMD:R_0805_2012Metric, symbol Device:R_US
- R25: value R_US -> 1k; footprint (none) -> Resistor_SMD:R_0805_2012Metric; MFG (none) -> YAGEO; MPN (none) -> RC0805FR-131KL
- renumbered R26 to R27, R27 to R28, R28 to R29, R29 to R30, R30 to R31, R31 to R32, R32 to R33
Connections:
- net CCMCTRL: now also Q2.1 (G)
- net GND: now also Q2.2 (D), Q3.3 (S), Q4.3 (S)
- net GREEN_LED: now also Q3.2 (D)
- net RED_LED: now also Q4.2 (D)
- net at R25.2: now also R26.1; no longer D4.2 (A)
- net at T1.1 (Pin_1), U8.3 (Q): now also Q4.1 (G)
- net at D3.1 (K), D4.1 (K), R29.1: now also Q3.1 (G)
- new net: D4.2 (A), Q2.3 (S), R26.2

Commit message: rough layout done
Parts:
- removed T1: Test555, Connector_PinHeader_1.00mm:PinHeader_1x01_P1.00mm_Vertical, symbol Connector:Conn_01x01_Pin
- added R34: 22k, Resistor_SMD:R_0805_2012Metric, symbol Device:R_US
- R30: value 22k -> 10k
Connections:
- net GND: now also R34.2
- net at D3.1 (K), D4.1 (K), Q3.1 (G)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: now also R34.1
Changed lines of the file:
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@@
+	)
+	(junction
+		(at 100.584 62.23)
+		(diameter 0)
+		(color 0 0 0 0)
 	)
 	(junction
@@
 	)
 	(junction
-		(at 204.47 62.23)
-		(diameter 0)
-		(color 0 0 0 0)
-	)
-	(junction
 		(at 146.05 54.61)
 		(diameter 0)
@@
 	(wire
 		(pts
+			(xy 100.584 62.23) (xy 107.95 62.23)
+		)
+		(stroke
+			(width 0)
+			(type default)
+		)
+	)
+	(wire
+		(pts
 			(xy 207.01 81.28) (xy 207.01 41.91)
 		)
@@
 	(wire
 		(pts
-			(xy 82.55 62.23) (xy 107.95 62.23)
+			(xy 82.55 62.23) (xy 100.584 62.23)
 		)
 		(stroke
@@
 	(wire
 		(pts
-			(xy 204.47 49.53) (xy 204.47 62.23)
-		)
-		(stroke
-			(width 0)
-			(type default)
-		)
-	)
-	(wire
-		(pts
 			(xy 101.6 48.26) (xy 101.6 50.8)
 		)
@@
 	(wire
 		(pts
-			(xy 204.47 62.23) (xy 209.55 62.23)
+			(xy 201.93 62.23) (xy 209.55 62.23)
 		)
 		(stroke
@@
 	(wire
 		(pts
-			(xy 201.93 62.23) (xy 204.47 62.23)
-		)
-		(stroke
-			(width 0)
-			(type default)
-		)
-	)
-	(wire
-		(pts
 			(xy 156.21 55.88) (xy 156.21 78.74)
 		)
@@
 		(pts
 			(xy 189.23 77.47) (xy 189.23 88.9)
-		)
-		(stroke
-			(width 0)
-			(type default)
-		)
-	)
-	(wire
-		(pts
-			(xy 201.93 49.53) (xy 204.47 49.53)
 		)
 		(stroke
@@
 	(symbol
 		(lib_id "Device:R_US")
+		(at 125.73 46.99 0)
+		(unit 1)
+		(exclude_from_sim no)
+		(in_bom yes)
+		(on_board yes)
+		(dnp no)
+		(property "Reference" "R30"
+			(at 128.27 45.7199 0)
+			(effects
+				(font
+					(size 1.27 1.27)
+				)
+				(justify left)
+			)
+		)
+		(property "Value" "10k"
+			(at 128.27 48.2599 0)
+			(effects
+				(font
+					(size 1.27 1.27)
+				)
+				(justify left)
+			)
+		)
+		(property "Footprint" "Resistor_SMD:R_0805_2012Metric"
+			(at 126.746 47.244 90)
+			(effects
+				(font
+					(size 1.27 1.27)
+				)
+				(hide yes)
+			)
+		)
+		(property "Datasheet" "~"
+			(at 125.73 46.99 0)
+			(effects
+				(font
+					(size 1.27 1.27)
+				)
+				(hide yes)
+			)
+		)
+		(property "Description" "Resistor, US symbol"
+			(at 125.73 46.99 0)
+			(effects
+				(font
+					(size 1.27 1.27)
+				)
+				(hide yes)
+			)
+		)
+		(pin "1"
+		)
+		(pin "2"
+		)
+		(instances
+			(project "SafetyBoard"
+				(path "/30d029c6-868b-41ac-953d-167a7d76c1a3/83cb6a8b-0a8f-42f4-832f-715c5e86ba97"
+					(reference "R30")
+					(unit 1)
+				)
+			)
+		)
+	)
+	(symbol
+		(lib_id "Device:R_US")
 		(at 106.68 50.8 90)
 		(unit 1)
@@
 				(path "/30d029c6-868b-41ac-953d-167a7d76c1a3/83cb6a8b-0a8f-42f4-832f-715c5e86ba97"
 					(reference "R25")
+					(unit 1)
+				)
+			)
+		)
+	)
+	(symbol
+		(lib_id "power:GND")
+		(at 100.584 69.85 0)
+		(unit 1)
+		(exclude_from_sim no)
+		(in_bom yes)
+		(on_board yes)
+		(dnp no)
+		(property "Reference" "#PWR0100"
+			(at 100.584 76.2 0)
+			(effects
+				(font
+					(size 1.27 1.27)
+				)
+				(hide yes)
+			)
+		)
+		(property "Value" "GND"
+			(at 104.394 71.1199 0)
+			(effects
+				(font
+					(size 1.27 1.27)
+				)
+				(justify left)
+			)
+		)
+		(property "Footprint" ""
+			(at 100.584 69.85 0)
+			(effects
+				(font
+					(size 1.27 1.27)
+				)
+				(hide yes)
+			)
+		)
+		(property "Datasheet" ""
+			(at 100.584 69.85 0)
+			(effects
+				(font
+					(size 1.27 1.27)
+				)
+				(hide yes)
+			)
+		)
+		(property "Description" "Power symbol creates a global label with name \"GND\" , ground"
+			(at 100.584 69.85 0)
+			(effects
+				(font
+					(size 1.27 1.27)
+				)
+				(hide yes)
+			)
+		)
+		(pin "1"
+		)
+		(instances
+			(project "SafetyBoard"
+				(path "/30d029c6-868b-41ac-953d-167a7d76c1a3/83cb6a8b-0a8f-42f4-832f-715c5e86ba97"
+					(reference "#PWR0100")
 					(unit 1)
 				)
@@
 	)
 	(symbol
-		(lib_id "Connector:Conn_01x01_Pin")
-		(at 196.85 49.53 0)
-		(unit 1)
-		(exclude_from_sim no)
-		(in_bom yes)
-		(on_board yes)
-		(dnp no)
-		(fields_autoplaced yes)
-		(property "Reference" "T1"
-			(at 197.485 44.45 0)
-			(effects
-				(font
-					(size 1.27 1.27)
-				)
-			)
-		)
-		(property "Value" "Test555"
-			(at 197.485 46.99 0)
-			(effects
-				(font
-					(size 1.27 1.27)
-				)
-			)
-		)
-		(property "Footprint" "Connector_PinHeader_1.00mm:PinHeader_1x01_P1.00mm_Vertical"
-			(at 196.85 49.53 0)
-			(effects
-				(font
-					(size 1.27 1.27)
-				)
-				(hide yes)
-			)
-		)
-		(property "Datasheet" "~"
-			(at 196.85 49.53 0)
-			(effects
-				(font
-					(size 1.27 1.27)
-				)
-				(hide yes)
-			)
-		)
-		(property "Description" "Generic connector, single row, 01x01, script generated"
-			(at 196.85 49.53 0)
-			(effects
-				(font
-					(size 1.27 1.27)
-				)
-				(hide yes)
-			)
-		)
-		(pin "1"
-		)
-		(instances
-			(project "TSSI2026.3"
-				(path "/30d029c6-868b-41ac-953d-167a7d76c1a3/83cb6a8b-0a8f-42f4-832f-715c5e86ba97"
-					(reference "T1")
-					(unit 1)
-				)
-			)
-			(project "TSSI2026.3"
-				(path "/9d68cf00-7b78-45a1-9a66-0d88bd9188eb"
-					(reference "T555")
-					(unit 1)
-				)
-			)
-		)
-	)
-	(symbol
 		(lib_id "Transistor_FET:IRLIZ44N")
 		(at 123.19 62.23 0)
@@
 				(path "/30d029c6-868b-41ac-953d-167a7d76c1a3/83cb6a8b-0a8f-42f4-832f-715c5e86ba97"
 					(reference "Q3")
-					(unit 1)
-				)
-			)
-		)
-	)
-	(symbol
-		(lib_id "Device:R_US")
-		(at 125.73 46.99 0)
-		(unit 1)
-		(exclude_from_sim no)
-		(in_bom yes)
-		(on_board yes)
-		(dnp no)
-		(property "Reference" "R30"
-			(at 127.508 45.72 0)
-			(effects
-				(font
-					(size 1.27 1.27)
-				)
-				(justify left)
-			)
-		)
-		(property "Value" "22k"
-			(at 127.508 48.26 0)
-			(effects
-				(font
-					(size 1.27 1.27)
-				)
-				(justify left)
-			)
-		)
-		(property "Footprint" "Resistor_SMD:R_0805_2012Metric"
-			(at 126.746 47.244 90)
-			(effects
-				(font
-					(size 1.27 1.27)
-				)
-				(hide yes)
-			)
-		)
-		(property "Datasheet" "~"
-			(at 125.73 46.99 0)
-			(effects
-				(font
-					(size 1.27 1.27)
-				)
-				(hide yes)
-			)
-		)
-		(property "Description" "Resistor, US symbol"
-			(at 125.73 46.99 0)
-			(effects
-				(font
-					(size 1.27 1.27)
-				)
-				(hide yes)
-			)
-		)
-		(pin "1"
-		)
-		(pin "2"
-		)
-		(instances
-			(project "TSSI2026.3"
-				(path "/30d029c6-868b-41ac-953d-167a7d76c1a3/83cb6a8b-0a8f-42f4-832f-715c5e86ba97"
-					(reference "R30")
-					(unit 1)
-				)
-			)
-			(project "TSSI2026.3"
-				(path "/9d68cf00-7b78-45a1-9a66-0d88bd9188eb"
-					(reference "R1")
 					(unit 1)
 				)
@@
 					(unit 1)
 				)
+			)
+		)
+	)
+	(symbol
+		(lib_id "Device:R_US")
+		(at 100.584 66.04 0)
+		(unit 1)
+		(exclude_from_sim no)
+		(in_bom yes)
+		(on_board yes)
+		(dnp no)
+		(property "Reference" "R34"
+			(at 102.362 64.77 0)
+			(effects
+				(font
+					(size 1.27 1.27)
+				)
+				(justify left)
+			)
+		)
+		(property "Value" "22k"
+			(at 102.362 67.31 0)
+			(effects
+				(font
+					(size 1.27 1.27)
+				)
+				(justify left)
+			)
+		)
+		(property "Footprint" "Resistor_SMD:R_0805_2012Metric"
+			(at 101.6 66.294 90)
+			(effects
+				(font
+					(size 1.27 1.27)
+				)
+				(hide yes)
+			)
+		)
+		(property "Datasheet" "~"
+			(at 100.584 66.04 0)
+			(effects
+				(font
+					(size 1.27 1.27)
+				)
+				(hide yes)
+			)
+		)
+		(property "Description" "Resistor, US symbol"
+			(at 100.584 66.04 0)
+			(effects
+				(font
+					(size 1.27 1.27)
+				)
+				(hide yes)
+			)
+		)
+		(pin "1"
+		)
+		(pin "2"
+		)
+		(instances
+			(project "SafetyBoard"
+				(path "/30d029c6-868b-41ac-953d-167a7d76c1a3/83cb6a8b-0a8f-42f4-832f-715c5e86ba97"
+					(reference "R34")
+					(unit 1)
+				)
