File: TSSI/TSSI/TSSI.kicad_sch (KiCad schematic)
At the start: 25 parts, among them J9 TSSI, Q2 IRLIZ44N NMOS, Q3 IRLIZ44N NMOS, Q4 IRLIZ44N NMOS, U8 LM555xN

Commit message: I think think this is final but need to defuck the BOM
Parts:
- removed D5: ON when ok, LED_THT:LED_D5.0mm, symbol Device:LED
- added D4: ON when ok, LED_THT:LED_D5.0mm, symbol Device:LED
- renumbered D3 to D2, D4 to D3, J9 to J10, R25 to R26, R26 to R27, R27 to R28, R34 to R29, R28 to R30, R29 to R31, R30 to R32, R31 to R33, R32 to R34, R33 to R35
Connections:
- net GND: now also D4.1 (K)
- net at R31.2: now also D4.2 (A)
Changed lines of the file:
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@@
 		(dnp no)
 		(fields_autoplaced yes)
-		(property "Reference" "#PWR066"
+		(property "Reference" "#PWR068"
 			(at 125.73 80.01 0)
 			(effects
@@
 			(project "TSSI2026.3"
 				(path "/30d029c6-868b-41ac-953d-167a7d76c1a3/83cb6a8b-0a8f-42f4-832f-715c5e86ba97"
-					(reference "#PWR066")
+					(reference "#PWR068")
 					(unit 1)
 				)
@@
 		(dnp no)
 		(fields_autoplaced yes)
-		(property "Reference" "D4"
+		(property "Reference" "D3"
 			(at 84.836 64.7699 90)
 			(effects
@@
 			(project "SafetyBoard"
 				(path "/30d029c6-868b-41ac-953d-167a7d76c1a3/83cb6a8b-0a8f-42f4-832f-715c5e86ba97"
-					(reference "D4")
+					(reference "D3")
 					(unit 1)
 				)
@@
 		(on_board yes)
 		(dnp no)
-		(property "Reference" "R27"
+		(property "Reference" "R28"
 			(at 95.25 49.022 0)
 			(effects
@@
 			(project "TSSI2026.3"
 				(path "/30d029c6-868b-41ac-953d-167a7d76c1a3/83cb6a8b-0a8f-42f4-832f-715c5e86ba97"
-					(reference "R27")
+					(reference "R28")
 					(unit 1)
 				)
@@
 		(on_board yes)
 		(dnp no)
-		(property "Reference" "R30"
+		(property "Reference" "R32"
 			(at 128.27 45.7199 0)
 			(effects
@@
 			(project "SafetyBoard"
 				(path "/30d029c6-868b-41ac-953d-167a7d76c1a3/83cb6a8b-0a8f-42f4-832f-715c5e86ba97"
-					(reference "R30")
+					(reference "R32")
 					(unit 1)
 				)
@@
 		(on_board yes)
 		(dnp no)
-		(property "Reference" "R28"
+		(property "Reference" "R30"
 			(at 105.41 49.022 0)
 			(effects
@@
 			(project "TSSI2026.3"
 				(path "/30d029c6-868b-41ac-953d-167a7d76c1a3/83cb6a8b-0a8f-42f4-832f-715c5e86ba97"
-					(reference "R28")
+					(reference "R30")
 					(unit 1)
 				)
@@
 		(on_board yes)
 		(dnp no)
-		(property "Reference" "#PWR063"
+		(property "Reference" "#PWR064"
 			(at 60.198 98.298 0)
 			(effects
@@
 			(project "SafetyBoard"
 				(path "/30d029c6-868b-41ac-953d-167a7d76c1a3/83cb6a8b-0a8f-42f4-832f-715c5e86ba97"
-					(reference "#PWR063")
+					(reference "#PWR064")
 					(unit 1)
 				)
@@
 		(dnp no)
 		(fields_autoplaced yes)
-		(property "Reference" "R25"
+		(property "Reference" "R26"
 			(at 62.992 66.5479 0)
 			(effects
@@
 			(project "SafetyBoard"
 				(path "/30d029c6-868b-41ac-953d-167a7d76c1a3/83cb6a8b-0a8f-42f4-832f-715c5e86ba97"
-					(reference "R25")
+					(reference "R26")
 					(unit 1)
 				)
@@
 		(on_board yes)
 		(dnp no)
-		(property "Reference" "#PWR0100"
+		(property "Reference" "#PWR065"
 			(at 100.584 76.2 0)
 			(effects
@@
 			(project "SafetyBoard"
 				(path "/30d029c6-868b-41ac-953d-167a7d76c1a3/83cb6a8b-0a8f-42f4-832f-715c5e86ba97"
-					(reference "#PWR0100")
+					(reference "#PWR065")
 					(unit 1)
 				)
@@
 		(on_board yes)
 		(dnp no)
-		(property "Reference" "#PWR064"
+		(property "Reference" "#PWR066"
 			(at 107.95 83.82 0)
 			(effects
@@
 			(project "TSSI2026.3"
 				(path "/30d029c6-868b-41ac-953d-167a7d76c1a3/83cb6a8b-0a8f-42f4-832f-715c5e86ba97"
-					(reference "#PWR064")
+					(reference "#PWR066")
 					(unit 1)
 				)
@@
 		(on_board yes)
 		(dnp no)
-		(property "Reference" "#PWR065"
+		(property "Reference" "#PWR067"
 			(at 110.49 57.15 0)
 			(effects
@@
 			(project "TSSI2026.3"
 				(path "/30d029c6-868b-41ac-953d-167a7d76c1a3/83cb6a8b-0a8f-42f4-832f-715c5e86ba97"
-					(reference "#PWR065")
+					(reference "#PWR067")
 					(unit 1)
 				)
@@
 		(on_board yes)
 		(dnp no)
-		(property "Reference" "R32"
+		(property "Reference" "R34"
 			(at 161.798 73.914 90)
 			(effects
@@
 			(project "TSSI2026.3"
 				(path "/30d029c6-868b-41ac-953d-167a7d76c1a3/83cb6a8b-0a8f-42f4-832f-715c5e86ba97"
-					(reference "R32")
+					(reference "R34")
 					(unit 1)
 				)
@@
 		(on_board yes)
 		(dnp no)
-		(property "Reference" "R33"
+		(property "Reference" "R35"
 			(at 219.71 45.7199 0)
 			(effects
@@
 			(project "TSSI2026.3"
 				(path "/30d029c6-868b-41ac-953d-167a7d76c1a3/83cb6a8b-0a8f-42f4-832f-715c5e86ba97"
-					(reference "R33")
+					(reference "R35")
 					(unit 1)
 				)
@@
 	)
 	(symbol
+		(lib_id "Device:LED")
+		(at 107.95 73.66 90)
+		(unit 1)
+		(exclude_from_sim no)
+		(in_bom yes)
+		(on_board yes)
+		(dnp no)
+		(fields_autoplaced yes)
+		(property "Reference" "D4"
+			(at 111.76 73.9774 90)
+			(effects
+				(font
+					(size 1.27 1.27)
+				)
+				(justify right)
+			)
+		)
+		(property "Value" "ON when ok"
+			(at 111.76 76.5174 90)
+			(effects
+				(font
+					(size 1.27 1.27)
+				)
+				(justify right)
+			)
+		)
+		(property "Footprint" "LED_THT:LED_D5.0mm"
+			(at 107.95 73.66 0)
+			(effects
+				(font
+					(size 1.27 1.27)
+				)
+				(hide yes)
+			)
+		)
+		(property "Datasheet" "~"
+			(at 107.95 73.66 0)
+			(effects
+				(font
+					(size 1.27 1.27)
+				)
+				(hide yes)
+			)
+		)
+		(property "Description" "Light emitting diode"
+			(at 107.95 73.66 0)
+			(effects
+				(font
+					(size 1.27 1.27)
+				)
+				(hide yes)
+			)
+		)
+		(property "Sim.Pins" "1=K 2=A"
+			(at 107.95 73.66 0)
+			(effects
+				(font
+					(size 1.27 1.27)
+				)
+				(hide yes)
+			)
+		)
+		(pin "1"
+		)
+		(pin "2"
+		)
+		(instances
+			(project "SafetyBoard"
+				(path "/30d029c6-868b-41ac-953d-167a7d76c1a3/83cb6a8b-0a8f-42f4-832f-715c5e86ba97"
+					(reference "D4")
+					(unit 1)
+				)
+			)
+		)
+	)
+	(symbol
 		(lib_id "Device:R_US")
 		(at 60.198 75.438 0)
@@
 		(dnp no)
 		(fields_autoplaced yes)
-		(property "Reference" "R26"
+		(property "Reference" "R27"
 			(at 62.23 74.1679 0)
 			(effects
@@
 			(project "SafetyBoard"
 				(path "/30d029c6-868b-41ac-953d-167a7d76c1a3/83cb6a8b-0a8f-42f4-832f-715c5e86ba97"
-					(reference "R26")
+					(reference "R27")
 					(unit 1)
 				)
@@
 		(on_board yes)
 		(dnp no)
-		(property "Reference" "R31"
+		(property "Reference" "R33"
 			(at 157.988 48.26 0)
 			(effects
@@
 			(project "TSSI2026.3"
 				(path "/30d029c6-868b-41ac-953d-167a7d76c1a3/83cb6a8b-0a8f-42f4-832f-715c5e86ba97"
-					(reference "R31")
+					(reference "R33")
 					(unit 1)
 				)
@@
 	)
 	(symbol
-		(lib_id "Device:LED")
-		(at 107.95 73.66 90)
-		(unit 1)
-		(exclude_from_sim no)
-		(in_bom yes)
-		(on_board yes)
-		(dnp no)
-		(fields_autoplaced yes)
-		(property "Reference" "D5"
-			(at 111.76 73.9774 90)
-			(effects
-				(font
-					(size 1.27 1.27)
-				)
-				(justify right)
-			)
-		)
-		(property "Value" "ON when ok"
-			(at 111.76 76.5174 90)
-			(effects
-				(font
-					(size 1.27 1.27)
-				)
-				(justify right)
-			)
-		)
-		(property "Footprint" "LED_THT:LED_D5.0mm"
-			(at 107.95 73.66 0)
-			(effects
-				(font
-					(size 1.27 1.27)
-				)
-				(hide yes)
-			)
-		)
-		(property "Datasheet" "~"
-			(at 107.95 73.66 0)
-			(effects
-				(font
-					(size 1.27 1.27)
-				)
-				(hide yes)
-			)
-		)
-		(property "Description" "Light emitting diode"
-			(at 107.95 73.66 0)
-			(effects
-				(font
-					(size 1.27 1.27)
-				)
-				(hide yes)
-			)
-		)
-		(property "Sim.Pins" "1=K 2=A"
-			(at 107.95 73.66 0)
-			(effects
-				(font
-					(size 1.27 1.27)
-				)
-				(hide yes)
-			)
-		)
-		(pin "1"
-		)
-		(pin "2"
-		)
-		(instances
-			(project "SafetyBoard"
-				(path "/30d029c6-868b-41ac-953d-167a7d76c1a3/83cb6a8b-0a8f-42f4-832f-715c5e86ba97"
-					(reference "D5")
-					(unit 1)
-				)
-			)
-		)
-	)
-	(symbol
 		(lib_name "MountingHole_1")
 		(lib_id "Mechanical:MountingHole")
@@
 		(on_board yes)
 		(dnp no)
-		(property "Reference" "J9"
+		(property "Reference" "J10"
 			(at 29.464 32.004 0)
 			(effects
@@
 			(project "SafetyBoard"
 				(path "/30d029c6-868b-41ac-953d-167a7d76c1a3/83cb6a8b-0a8f-42f4-832f-715c5e86ba97"
-					(reference "J9")
+					(reference "J10")
 					(unit 1)
 				)
@@
 		(dnp no)
 		(fields_autoplaced yes)
-		(property "Reference" "#PWR068"
+		(property "Reference" "#PWR070"
 			(at 217.17 99.06 0)
 			(effects
@@
 			(project "TSSI2026.3"
 				(path "/30d029c6-868b-41ac-953d-167a7d76c1a3/83cb6a8b-0a8f-42f4-832f-715c5e86ba97"
-					(reference "#PWR068")
+					(reference "#PWR070")
 					(unit 1)
 				)
@@
 		(on_board yes)
 		(dnp no)
-		(property "Reference" "R34"
+		(property "Reference" "R29"
 			(at 102.362 64.77 0)
 			(effects
@@
 			(project "SafetyBoard"
 				(path "/30d029c6-868b-41ac-953d-167a7d76c1a3/83cb6a8b-0a8f-42f4-832f-715c5e86ba97"
-					(reference "R34")
+					(reference "R29")
 					(unit 1)
 				)
@@
 		(dnp no)
 		(fields_autoplaced yes)
-		(property "Reference" "#PWR067"
+		(property "Reference" "#PWR069"
 			(at 189.23 99.06 0)
 			(effects
@@
 			(project "TSSI2026.3"
 				(path "/30d029c6-868b-41ac-953d-167a7d76c1a3/83cb6a8b-0a8f-42f4-832f-715c5e86ba97"
-					(reference "#PWR067")
+					(reference "#PWR069")
 					(unit 1)
 				)
@@
 		(on_board yes)
 		(dnp no)
-		(property "Reference" "R29"
+		(property "Reference" "R31"
 			(at 109.728 64.77 0)
 			(effects
@@
 			(project "TSSI2026.3"
 				(path "/30d029c6-868b-41ac-953d-167a7d76c1a3/83cb6a8b-0a8f-42f4-832f-715c5e86ba97"
-					(reference "R29")
+					(reference "R31")
 					(unit 1)
 				)
@@
 		(dnp no)
 		(fields_autoplaced yes)
-		(property "Reference" "D3"
+		(property "Reference" "D2"
 			(at 85.09 53.3399 90)
 			(effects
@@
 			(project "SafetyBoard"
 				(path "/30d029c6-868b-41ac-953d-167a7d76c1a3/83cb6a8b-0a8f-42f4-832f-715c5e86ba97"
-					(reference "D3")
-					(unit 1)
-				)
+					(reference "D2")
+					(unit 1)
+				)

Commit message: updates I think
Parts:
- removed H5, H6, H7, H8: MountingHole, MountingHole:MountingHole_3.2mm_M3, symbol Mechanical:MountingHole
