File: 2026CCM/ccm.kicad_sch (KiCad schematic)
At the start: 102 parts, among them J1 Conn_01x02_Socket, J10 Conn_01x02_Socket, J11 Conn_01x02_Socket, J12 Conn_01x02_Socket, J13 Conn_01x02_Socket, J14 Conn_01x04_Socket, J15 Conn_01x02_Socket, J16 Conn_01x04_Socket, J17 Conn_01x04_Socket, J18 Conn_01x04_Socket, J19 Conn_01x02_Socket, J2 Conn_01x02_Socket, J20 Conn_01x02_Socket, J21 Conn_01x02_Socket, J3 Conn_01x02_Socket, J4 Conn_01x04_Socket, J5 Conn_01x04_Socket, J6 Conn_01x02_Socket, J7 Conn_01x02_Socket, J8 Conn_01x04_Socket, J9 Conn_01x02_Socket, Q1 IRLZ34N, Q2 IRLZ34N, Q3 IRLZ34N, Q4 IRLZ34N, Q5 IRLZ34N, Q6 IRLZ34N, Q7 IRLZ34N, U1 Teensy4.1, U2 PAM8302AAY, U3 SN65HVD230, U4 SN65HVD230, U5 LM1117DT-5.0

Commit message: ccm v2.1
new speaker amp, fixed keyswitch control
Parts:
- removed R51: 10k, Resistor_SMD:R_0805_2012Metric, symbol Device:R
- removed U2: PAM8302AAY, Package_DFN_QFN:DFN-8-1EP_3x3mm_P0.65mm_EP1.55x2.4mm, symbol Amplifier_Audio:PAM8302AAY
- added C13: 10nF, Capacitor_SMD:C_0805_2012Metric, symbol Device:C
- added C14: 100nF, Capacitor_SMD:C_0805_2012Metric, symbol Device:C
- added C15, C16: 470nF, Capacitor_SMD:C_0805_2012Metric, symbol Device:C
- added C17, C18: 1uF, Capacitor_SMD:C_0805_2012Metric, symbol Device:C
- added D3, D4: ESD562DBZRQ1, ESD2CAN24DBZRQ1:SOT95P237X112-3N, symbol custom:ESD562DBZRQ1
- added R51: 1k, Resistor_SMD:R_0805_2012Metric, symbol Device:R_US
- added R52: 10, Resistor_SMD:R_0805_2012Metric, symbol Device:R_US
- added U6: TPA3111D1PWPR, PWP28_6P17X2P4, symbol custom:TPA3111D1PWPR
- C10: value 10nF -> 1nF
- C7: value 0.1uF -> 100nF
- C8: value 1uF -> 1nF
- C9: value 10uF -> 100nF
- R23: value 1k -> 100k
Connections:
- net +5V: no longer C8.1, C9.1
- net CANH_1: now also D3.2
- net CANH_2: now also D4.2
- net CANL_1: now also D3.1
- net CANL_2: now also D4.1
- net GLV-: now also C10.2, C7.2, C13.2, C17.1, C18.2, D3.3, D4.3, U6.11 (INN), U6.19 (PGND), U6.24 (PGND), U6.29 (EPAD), U6.3 (GND), U6.4 (GND), U6.5 (GAIN0), U6.6 (GAIN1), U6.8 (AGND); no longer C10.1
- net Vin: now also C10.1, C7.1, C8.1, C9.1, Q6.2 (D), R23.2, R52.1, U6.15 (PVCC), U6.16 (PVCC), U6.27 (PVCC), U6.28 (PVCC)
- net speaker+: now also C16.1, U6.18 (OUTP), U6.20 (OUTP)
- net speaker-: now also C15.1, U6.23 (OUTN), U6.25 (OUTN)
- net speaker_pwm: now also R51.1; no longer R23.2
- new net: C16.2, U6.17 (BSP), U6.21 (BSP)
- new net: R23.1, U6.1 (*SD), U6.2 (*FAULT)
- new net: C17.2, R52.2, U6.14 (AVCC), U6.7 (AVCC)
- new net: C18.1, U6.10 (PLIMIT), U6.9 (GVDD)
- new net: C14.2, U6.12 (INP)
- new net: C15.2, U6.22 (BSN), U6.26 (BSN)
- new net: C13.1, C14.1, R51.2
Other:
- moved on the sheet: C1, C2, C5, R25, R27, R28, R29, R3, R30, R31, R32, U3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
