File: BSPD/BSPD/BSPD.kicad_sch (KiCad schematic)
At the start: 75 parts, among them J1 T2M-105-01-X-D-TH-DS, J2 39-30-6068, Q1 IRLIZ44N NMOS, U1 LM393, U2 4071 4 Channel 2 Input OR gate, U3 LM393, U4 LM393, U5 4081 AND Gate, U6 40106 Inverter

Commit message: Changed a buncha stuff on other ppl's board. established new branch
Parts:
- removed J1: T2M-105-01-X-D-TH-DS, T2M_105:SAMTEC_T2M-105-01-X-D-TH-DS, symbol T2M-105-01-X-D-TH-DS:T2M-105-01-X-D-TH-DS
- removed J2: 39-30-6068, 39-30:39-30-606Y, symbol 39-30-6068:39-30-6068
- renumbered C8 to C1, C3 to C10, C10 to C2, C9 to C3, C7 to C4, C6 to C5, C1 to C6, C2 to C7, C4 to C8, C5 to C9, D2 to D1, D1 to D2, H4 to H3, H3 to H4, R21 to R1, R7 to R10, R6 to R11, R10 to R12, R8 to R13, R16 to R14, R17 to R15, R5 to R16, R1 to R17, R4 to R18, R11 to R19, R18 to R2, R13 to R20, R14 to R21, R15 to R22, R9 to R23, R12 to R24, R20 to R3, R22 to R4, R19 to R5, R24 to R6, R23 to R7, R2 to R8, R3 to R9, TP16 to TP1, TP1 to TP10, TP3 to TP11, TP11 to TP12, TP17 to TP13, TP6 to TP14, TP4 to TP15, TP5 to TP16, TP13 to TP17, TP14 to TP2, TP10 to TP3, TP2 to TP4, TP8 to TP5, TP15 to TP6, TP9 to TP7, TP12 to TP8, TP7 to TP9, U6 to U1, U5 to U2, U1 to U3, U3 to U4, U2 to U5, U4 to U6
Connections:
- net BSPD_FAULT renamed BSPD Fault
- net B_IN renamed Brake Sensor
- net C_IN renamed Current Sensor
- no-connect marks 5 -> 4

Commit message: day 2 grind
Parts:
- added J8: Current Sensor, 0footprints:Molex_Mini-Fit_Jr_5566-04A_2x02_P4.20mm_Vertical, symbol Connector_Generic:Conn_02x02_Top_Bottom
- added U3: LT1084-5.0, Package_TO_SOT_THT:TO-220-3_Horizontal_TabDown, symbol Regulator_Linear:LT1084-5.0
- renumbered U3 to U4, U4 to U5, U5 to U6, U6 to U7
Connections:
- net +12V: now also U3.3 (VI)
- net GND: now also J8.4 (Pin_4), U3.1 (GND)
- net Current Sensor renamed C_IN
- net C_IN: now also J8.2 (Pin_2)
- new net +5V: J8.1 (Pin_1), U3.2 (VO)
- no-connect marks 4 -> 5

Commit message: hopefully this lets avadi pull
Parts:
- LED1, LED2, LED3: footprint SMALL_LED:LEDC2012X105N -> LED_SMD:LED_0805_2012Metric_Pad1.15x1.40mm_HandSolder
- Q1: footprint Package_TO_SOT_THT:TO-220F-3_Vertical -> Package_TO_SOT_THT:TO-220F-3_Horizontal_TabDown

Commit message: rough layout done
Parts:
- removed D1: D, Diode_SMD:D_0603_1608Metric, symbol Device:D
- removed TP1: BRAKE, TestPoint:TestPoint_Pad_D2.5mm, symbol Connector:TestPoint
- removed TP10: B_SHORT, TestPoint:TestPoint_Pad_D2.5mm, symbol Connector:TestPoint
- removed TP11: B_OPEN, TestPoint:TestPoint_Pad_D2.5mm, symbol Connector:TestPoint
- removed TP12: P_SHORT, TestPoint:TestPoint_Pad_D2.5mm, symbol Connector:TestPoint
- removed TP13: P_OPEN, TestPoint:TestPoint_Pad_D2.5mm, symbol Connector:TestPoint
- removed TP14: B_ERROR, TestPoint:TestPoint_Pad_D2.5mm, symbol Connector:TestPoint
- removed TP15: P_ERROR, TestPoint:TestPoint_Pad_D2.5mm, symbol Connector:TestPoint
- removed TP16: FAULT_SENSED, TestPoint:TestPoint_Pad_D2.5mm, symbol Connector:TestPoint
- removed TP17: BSPD_FAULT, TestPoint:TestPoint_Pad_D2.5mm, symbol Connector:TestPoint
- removed TP2: PEDAL, TestPoint:TestPoint_Pad_D2.5mm, symbol Connector:TestPoint
- removed TP3: SC, TestPoint:TestPoint_Pad_D2.5mm, symbol Connector:TestPoint
- removed TP4: OC, TestPoint:TestPoint_Pad_D2.5mm, symbol Connector:TestPoint
- removed TP5: BRAKE_TH, TestPoint:TestPoint_Pad_D2.5mm, symbol Connector:TestPoint
- removed TP6: PEDAL_TH, TestPoint:TestPoint_Pad_D2.5mm, symbol Connector:TestPoint
- removed TP7: B_APPLIED, TestPoint:TestPoint_Pad_D2.5mm, symbol Connector:TestPoint
- removed TP8: P_APPLIED, TestPoint:TestPoint_Pad_D2.5mm, symbol Connector:TestPoint
- removed TP9: BOTH_ON, TestPoint:TestPoint_Pad_D2.5mm, symbol Connector:TestPoint
Other:
- note removed: "Test Points"

Commit message: silkscreen and some fuses or something
Parts:
- U6: value 4071 4 Channel 2 Input OR gate -> CD4071BE OR Gate
Changed lines of the file:
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@@
 			)
 		)
-		(property "Value" "4071 4 Channel 2 Input OR gate"
+		(property "Value" "CD4071BE OR Gate"
 			(at 298.704 192.278 0)
 			(effects
@@
 					(size 1.27 1.27)
 				)
-				(hide yes)
 			)
 		)
@@
 			)
 		)
-		(property "Value" "4071 4 Channel 2 Input OR gate"
+		(property "Value" "CD4071BE OR Gate"
 			(at 381 224.028 0)
 			(effects
@@
 			)
 		)
-		(property "Value" "4071 4 Channel 2 Input OR gate"
+		(property "Value" "CD4071BE OR Gate"
 			(at 381 214.376 0)
 			(effects
@@
 			)
 		)
-		(property "Value" "4071 4 Channel 2 Input OR gate"
+		(property "Value" "CD4071BE OR Gate"
 			(at 295.91 210.82 0)
 			(effects
@@
 			)
 		)
-		(property "Value" "4071 4 Channel 2 Input OR gate"
+		(property "Value" "CD4071BE OR Gate"
 			(at 337.82 200.66 0)
 			(effects

Commit message: I think think this is final but need to defuck the BOM
Parts:
- added R12: 10k, Resistor_SMD:R_0603_1608Metric, symbol Device:R
- renumbered LED3 to BothThreshold1, D2 to D1, J8 to J9, LED2 to OutOfRange1, R12 to R13, R13 to R14, R14 to R15, R15 to R16, R16 to R17, R17 to R18, R18 to R19, R19 to R20, R20 to R21, R21 to R22, R22 to R23, R23 to R24, R24 to R25, R_Bypass1 to SchmittDis1, LED1 to brkErr1, R_Bypass2 to schmittEN1
Connections:
- net FAULT_SENSED: now also R12.1
- net GND: now also R12.2
