File: ChargerBoard/ChargeBoard/ChargeBoardMaster.kicad_pcb (KiCad board)
At the start: 2 copper layers, 123 x 120.7 mm, 40 parts, among them J1 DT15-12PA, J2 ESTOP, J3 HVIL, J4 to Lead Acid Batt, J5 BatteryTender, J7 J1772, J8 874271042, K1 G6B-2214P-US DC12, K2 G6B-2214P-US DC12, Q1 PMOS IRF9540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

Commit message: silkscreen, last touches time to order
Other:
- board text added: "Charger PCB By Gabriel Schoene"
