File: ChargerBoard/ChargeBoard/ChargeBoardMaster.kicad_sch (KiCad schematic)
At the start: 23 parts, among them J1 DT15-12PA, J2 ESTOP, J3 HVIL, J4 to Lead Acid Batt, J5 BatteryTender, J7 J1772, J8 874271042

Commit message: silkscreen, last touches time to order
Parts:
- R9: value 120r -> 60r
Changed lines of the file:
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@@
 		(fields_autoplaced yes)
 		(property "Reference" "R9"
-			(at 113.538 140.2079 0)
+			(at 113.03 140.2079 0)
 			(effects
 				(font
@@
 			)
 		)
-		(property "Value" "120r"
-			(at 113.538 142.7479 0)
+		(property "Value" "60r"
+			(at 113.03 142.7479 0)
 			(effects
 				(font

Commit message: whoops forgot can on charger board
Parts:
- R9: value 60r -> 120r
Connections:
- net CANH: now also J1.6
- net CANL: now also J1.7
- no-connect marks 5 -> 3
Other:
- moved on the sheet: J7
Changed lines of the file:
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@@
-	)
-	(no_connect
-		(at 37.592 141.478)
-	)
-	(no_connect
-		(at 37.592 138.938)
 	)
 	(no_connect
@@
 	(wire
 		(pts
+			(xy 97.79 167.64) (xy 97.79 183.896)
+		)
+		(stroke
+			(width 0)
+			(type default)
+		)
+	)
+	(wire
+		(pts
 			(xy 162.56 60.452) (xy 161.036 60.452)
 		)
@@
 	(wire
 		(pts
-			(xy 103.124 183.896) (xy 97.282 183.896)
+			(xy 97.79 167.64) (xy 97.028 167.64)
 		)
 		(stroke
@@
 	(wire
 		(pts
-			(xy 90.424 183.896) (xy 94.742 183.896)
-		)
-		(stroke
-			(width 0)
-			(type default)
-		)
-	)
-	(wire
-		(pts
 			(xy 103.124 196.088) (xy 103.124 194.056)
 		)
@@
 	(wire
 		(pts
+			(xy 94.488 183.896) (xy 90.424 183.896)
+		)
+		(stroke
+			(width 0)
+			(type default)
+		)
+	)
+	(wire
+		(pts
+			(xy 97.79 183.896) (xy 103.124 183.896)
+		)
+		(stroke
+			(width 0)
+			(type default)
+		)
+	)
+	(wire
+		(pts
 			(xy 32.512 116.84) (xy 30.48 116.84)
+		)
+		(stroke
+			(width 0)
+			(type default)
+		)
+	)
+	(wire
+		(pts
+			(xy 94.488 167.64) (xy 94.488 183.896)
 		)
 		(stroke
@@
 		)
 	)
+	(label "CANH"
+		(at 37.592 138.938 180)
+		(effects
+			(font
+				(size 1.27 1.27)
+			)
+			(justify right bottom)
+		)
+	)
 	(label "IMD_FAULT"
 		(at 37.592 133.858 180)
@@
 	(label "LED_GND"
 		(at 140.97 143.002 180)
+		(effects
+			(font
+				(size 1.27 1.27)
+			)
+			(justify right bottom)
+		)
+	)
+	(label "CANL"
+		(at 37.592 141.478 180)
 		(effects
 			(font
@@
 	(symbol
 		(lib_id "2pMinifitJR:39310020")
-		(at 94.742 183.896 90)
+		(at 94.488 167.64 90)
 		(unit 1)
 		(exclude_from_sim no)
@@
 		(fields_autoplaced yes)
 		(property "Reference" "J7"
-			(at 100.584 173.7359 90)
+			(at 100.33 157.4799 90)
 			(effects
 				(font
@@
 		)
 		(property "Value" "J1772"
-			(at 100.584 176.2759 90)
+			(at 100.33 160.0199 90)
 			(effects
 				(font
@@
 		)
 		(property "Footprint" "MODELS:2pMinifitJR"
-			(at 94.742 183.896 0)
+			(at 94.488 167.64 0)
 			(effects
 				(font
@@
 		)
 		(property "Datasheet" "https://www.molex.com/en-us/products/part-detail-pdf/39310020?display=pdf"
-			(at 94.742 183.896 0)
+			(at 94.488 167.64 0)
 			(effects
 				(font
@@
 		)
 		(property "Description" ""
-			(at 94.742 183.896 0)
+			(at 94.488 167.64 0)
 			(effects
 				(font
@@
 		)
 		(property "MPN" "0469990138 "
-			(at 94.742 183.896 0)
+			(at 94.488 167.64 0)
 			(effects
 				(font
@@
 		)
 		(property "MFG" "Molex "
-			(at 94.742 183.896 0)
+			(at 94.488 167.64 0)
 			(effects
 				(font
@@
 			)
 		)
-		(property "Value" "60r"
+		(property "Value" "120r"
 			(at 113.03 142.7479 0)
 			(effects
