File: Precharge Control Circuit/PCC/PCC.kicad_pcb (KiCad board)
At the start: 2 copper layers, 190.6 x 151.7 mm, 137 parts, among them J1 Conn_01x04_Socket, J10 AMP BYP, J11 AMP BYP, J12 INVTR, J2 874271202, J3 462070206, J4 Conn_02x14_Counter_Clockwise, J5 IMD, J6 Thermistor Expansion, J7 RTM, J8 BMS, J9 EnergyMeter, K1 Relay_SPDT, K2 PCN-112D3MHZ_000, Q1 IRLZ44N, Q2 IRLZ44N, U1 SN65HVD230, U2 4N35, U3 4N35, U7 TLV2372IP, U8 LM1117T-5.0

Commit message: PCCv2 started
Parts:
- removed Charger1, DCDC1: 428192213, footprints:MOLEX_428192213
- removed D2: 1N4007, Diode_THT:D_DO-41_SOD81_P10.16mm_Horizontal
- removed F10, F11, F5, F6, F7, F8, F9: 1A, footprints:5x20fuseblock
- removed F12: 01220088Z, footprints:FuseHolder
- removed HVIN1: 428194213, footprints:MOLEX_428194213
- removed J7: RTM, Connector_Molex:Molex_Mini-Fit_Jr_5566-04A2_2x02_P4.20mm_Vertical
- removed K2: PCN-112D3MHZ_000, footprints:RELAY_PCN-105D3MHZ_000_TEC
- removed SDC2: Conn_01x02_Socket, Connector_Molex:Molex_Mini-Fit_Jr_5566-02A2_2x01_P4.20mm_Vertical
- added C27: 100nF, Capacitor_SMD:C_0805_2012Metric, F.Cu at (146.9, 98.1)
- added C28: 1uF, Capacitor_SMD:C_0805_2012Metric, B.Cu at (83.2, 130.1)
- added C29: 100nF, Capacitor_SMD:C_0805_2012Metric, B.Cu at (90.5, 136.5)
- added C30: 100nF, Capacitor_SMD:C_0805_2012Metric, B.Cu at (89.7, 128.9)
- added C31: 10u, Capacitor_SMD:C_0805_2012Metric, B.Cu at (105.8, 100.5)
- added C32: 100n, Capacitor_SMD:C_0805_2012Metric, B.Cu at (105.8, 103.5)
- added DEBUG_1: LED, LED_THT:LED_D5.0mm, F.Cu at (158.9, 109.2)
- added DEBUG_2: LED, LED_THT:LED_D5.0mm, F.Cu at (93.3, 123.5)
- added F1: 1A, footprints:5x20fuseblock, B.Cu at (164.2, 77.9)
- added F2: 1A, footprints:5x20fuseblock, F.Cu at (142.8, 106.8)
- added F3: 1A, footprints:5x20fuseblock, F.Cu at (130.7, 148.1)
- added F4: 1A, footprints:5x20fuseblock, F.Cu at (130.7, 159.6)
- added HS1: Heatsink_Pad, footprints:heatsink, F.Cu at (121.7, 83.9)
- added HS2: Heatsink_Pad, footprints:heatsink, F.Cu at (121.9, 130.9)
- added J13: 462070206, footprints:6pMinifitJR, F.Cu at (114.3, 150.4)
- added Q3: Q_NMOS_GSD, Package_TO_SOT_SMD:SOT-23, B.Cu at (105.7, 113.0)
- added Q4: Q_NMOS_GSD, Package_TO_SOT_SMD:SOT-23, B.Cu at (90.5, 118.6)
- added Q5: Q_NMOS_GSD, Package_TO_SOT_SMD:SOT-23, B.Cu at (78.5, 129.5)
- added R61: 510K, Resistor_SMD:R_0805_2012Metric, F.Cu at (122.2, 98.6)
- added R62: 20k, Resistor_SMD:R_0805_2012Metric, F.Cu at (128.0, 99.5)
- added R63: 510K, Resistor_SMD:R_0805_2012Metric, F.Cu at (122.7, 116.0)
- added R64: 20k, Resistor_SMD:R_0805_2012Metric, F.Cu at (126.8, 92.3)
- added R65: 510K, Resistor_SMD:R_0805_2012Metric, F.Cu at (122.8, 122.1)
- added R66: 20k, Resistor_SMD:R_0805_2012Metric, F.Cu at (122.5, 92.6)
- added R67: 510K, Resistor_SMD:R_0805_2012Metric, F.Cu at (127.2, 122.2)
- added R68: 20k, Resistor_SMD:R_0805_2012Metric, F.Cu at (159.2, 102.2)
- added R69: 510K, Resistor_SMD:R_0805_2012Metric, F.Cu at (128.0, 115.7)
- added R70: 10k, Resistor_SMD:R_0805_2012Metric, F.Cu at (108.0, 116.0)
- added R71: 20k, Resistor_SMD:R_0805_2012Metric, B.Cu at (90.6, 113.3)
- added R72: 20k, Resistor_SMD:R_0805_2012Metric, B.Cu at (86.8, 123.8)
- added R73: 22k, Resistor_SMD:R_0805_2012Metric, B.Cu at (87.6, 120.9)
- added R74: 22k, Resistor_SMD:R_0805_2012Metric, B.Cu at (89.9, 134.2)
- added R75: 220k, Resistor_SMD:R_0805_2012Metric, B.Cu at (89.9, 131.3)
- added R76: 11k, Resistor_SMD:R_0805_2012Metric, B.Cu at (115.6, 109.0)
- added R77: 10k, Resistor_SMD:R_0805_2012Metric, B.Cu at (77.5, 124.6)
- added R78: 0.43R 1/2W, Resistor_SMD:R_0805_2012Metric_Pad1.20x1.40mm_HandSolder, B.Cu at (163.8, 62.3)
- added R79: 0.43R 1/2W, Resistor_SMD:R_0805_2012Metric_Pad1.20x1.40mm_HandSolder, B.Cu at (132.8, 99.3)
- added R80: 0.43R 1/2W, Resistor_SMD:R_0805_2012Metric_Pad1.20x1.40mm_HandSolder, F.Cu at (146.6, 145.2)
- added R81: 0.43R 1/2W, Resistor_SMD:R_0805_2012Metric_Pad1.20x1.40mm_HandSolder, F.Cu at (146.8, 160.1)
- added RV1: 1k default (1-5k), Potentiometer_THT:Potentiometer_Bourns_3296Y_Vertical, F.Cu at (118.7, 101.6)
- added R_pullup1: 15k, Resistor_SMD:R_0805_2012Metric, B.Cu at (115.4, 112.3)
- added U10: 4N35, Package_DIP:DIP-6_W7.62mm, F.Cu at (101.2, 116.1)
- added U11: LM555xN, Package_DIP:DIP-8_W7.62mm, F.Cu at (86.2, 129.0)
- added U12: ~, footprints:isoDCDC(removedPins), F.Cu at (91.7, 107.0)
- added U9: TLV2372IP, footprints:P8, F.Cu at (120.1, 115.1)
- F13, F15, F16, F17: value 01220088Z -> 1A; footprint footprints:FuseHolder -> footprints:5x20fuseblock; moved to B.Cu
- F14, F18, F19: value 01220088Z -> 1A; footprint footprints:FuseHolder -> footprints:5x20fuseblock
- K1: footprint Relay_THT:Precharge_Discharge_Relay -> footprints:Precharge_Discharge_Relay_Rincon
- R3, R6: value 500 -> 2.7k; footprint footprints:Ohmite HS100 500R F -> Package_TO_SOT_THT:TO-220-2_Vertical
- moved R14 108.7 mm to (144.9, 31.2), turned to -90 degrees
- moved R15 105.1 mm to (146.6, 62.0)
- moved R6 104.0 mm to (119.2, 135.6), turned to 0 degrees
- moved J2 94.9 mm to (154.8, 34.2)
- moved R13 92.7 mm to (132.9, 115.5), turned to 180 degrees
- moved R18 92.4 mm to (151.2, 62.1), turned to 90 degrees
- moved R3 87.4 mm to (124.6, 79.3), turned to 180 degrees
- moved F13 78.3 mm to (142.8, 106.8)
- moved R19 76.8 mm to (159.6, 62.4), turned to 90 degrees
- moved R17 74.2 mm to (152.3, 29.4)
- moved R16 70.0 mm to (157.3, 48.6), turned to 90 degrees
- moved F18 68.3 mm to (151.8, 77.8), turned to 90 degrees
- moved H1 68.2 mm to (165.3, 21.6)
- moved H2 64.1 mm to (169.4, 157.8)
- moved F15 44.9 mm to (151.8, 77.8), turned to 90 degrees
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- renumbered J12 to J10, J10 to J11, J11 to J12
Connections:
- F13 pad 1: TS- -> TS+
- F13 pad 2: TS- -> Net-(F13-Pad2)
- F14 pad 1: TS+ -> TS-
- F14 pad 2: TS+ -> Net-(F14-Pad2)
- F15 pad 1: Net-(DCDC1-PadP1_1) -> TS+
- F15 pad 2: Net-(DCDC1-PadP1_1) -> Net-(F15-Pad2)
- F16 pad 1: TS+ -> TS-
- F16 pad 2: TS+ -> Net-(F16-Pad2)
- F17 pad 1: Net-(Charger1-PadP2_1) -> TS-
- F17 pad 2: Net-(Charger1-PadP2_1) -> Net-(F17-Pad2)
- F18 pad 1: Net-(Charger1-PadP1_1) -> TS+
- F18 pad 2: Net-(Charger1-PadP1_1) -> Net-(F18-Pad2)
- F19 pad 1: TS- -> TS+
- F19 pad 2: TS- -> Net-(F19-Pad2)
- J2 pad 1: /IL -> /FusedTS - (indicator)
- J2 pad 10: /FusedTS-3 -> unconnected-(J2-Pad10)
- J2 pad 11: unconnected-(J2-Pad11) -> /FusedTS + (expansion)
- J2 pad 12: /TSMP- -> /FusedTS + (IMD)
- J2 pad 2: /FusedTS+1 -> /TSMP-
- J2 pad 3: /FusedTS+2 -> /TSMP+
- J2 pad 4: /FusedTS+3 -> /FusedTS - (IMD)
- J2 pad 5: /FusedTS+4 -> /FusedTS+ (EM)
- J2 pad 6: /TSMP+ -> /FusedTS + (indicator)
- J2 pad 7: /IL -> /FusedTS - (expansion)
- J2 pad 8: /FusedTS-1 -> unconnected-(J2-Pad8)
- J2 pad 9: /FusedTS-2 -> unconnected-(J2-Pad9)
- K1 pad 12: TS- -> TS- unfused
- R1 pad 1: TS+ -> TS+ unfused
- R13 pad 1: Net-(F5-Pad2) -> Net-(F13-Pad2)
- R13 pad 2: /FusedTS+4 -> HighVoltage+
- R14 pad 1: Net-(F6-Pad2) -> Net-(F14-Pad2)
- R14 pad 2: /FusedTS-3 -> /FusedTS - (expansion)
- R15 pad 1: Net-(F7-Pad2) -> Net-(F15-Pad2)
- R15 pad 2: /FusedTS+3 -> /FusedTS + (expansion)
- R16 pad 1: Net-(F8-Pad2) -> Net-(F16-Pad2)
- R16 pad 2: /FusedTS-2 -> /FusedTS - (IMD)
- R17 pad 1: Net-(F9-Pad2) -> Net-(F17-Pad2)
- R17 pad 2: /FusedTS-1 -> /FusedTS - (indicator)
- R18 pad 1: Net-(F10-Pad2) -> Net-(F18-Pad2)
- R18 pad 2: /FusedTS+2 -> /FusedTS + (IMD)
- R19 pad 1: Net-(F11-Pad2) -> Net-(F19-Pad2)
- R19 pad 2: /FusedTS+1 -> /FusedTS + (indicator)
- R2 pad 1: TS- -> TS- unfused
- R3 pad 1: TS+ -> Net-(R3-Pad1)
- R3 pad 2: Net-(R3-Pad2) -> Vin_Accu
- R6 pad 1: Net-(R3-Pad2) -> TS+ unfused
- R6 pad 2: Vin_Accu -> Net-(R3-Pad1)
Routing:
- net TS+: track 308.9 -> 0.00 mm
- net TS-: track 173.4 -> 0.00 mm, vias 5 -> 0
- net B+_in: track 122.6 -> 15.7 mm, vias 1 -> 0
- net Vin_Accu: track 92.0 -> 0.00 mm
- net Net-(R3-Pad2): track 48.0 -> 0.00 mm
- net GND ISO: track 44.9 -> 0.00 mm, vias 1 -> 0
- net /TSMP+: track 42.8 -> 0.00 mm
- net Net-(U7-2IN+): track 44.8 -> 6.65 mm, vias 2 -> 0
- net /TSMP-: track 32.4 -> 0.00 mm
- net /FusedTS-1: track 28.4 -> 0.00 mm
- net Net-(U7-1IN+): track 35.8 -> 9.52 mm
- net TS+ unfused: track 0.00 -> 25.8 mm, vias 0 -> 1
- net TS- unfused: track 0.00 -> 22.0 mm, vias 0 -> 1
- net DCDC Enable B: track 17.8 -> 0.00 mm
- net Net-(F10-Pad2): track 15.7 -> 0.00 mm
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- removed copper zone on B.Cu, net Net-(Charger1-PadP1_1)
- removed copper zone on F.Cu, net Net-(Charger1-PadP1_1)
- removed copper zone on B.Cu, net Net-(Charger1-PadP2_1)
- removed copper zone on F.Cu, net Net-(Charger1-PadP2_1)
- removed copper zone on B.Cu, net Net-(DCDC1-PadP1_1)
- removed copper zone on F.Cu, net Net-(DCDC1-PadP1_1)
- removed copper zone on B.Cu, net Net-(DCDC1-PadP2_1)
- removed copper zone on F.Cu, net Net-(DCDC1-PadP2_1)
- removed copper zone on B.Cu, net Net-(R1-Pad2)
- removed copper zone on B.Cu, net Net-(R10-Pad1)
- removed copper zone on B.Cu, net Net-(R10-Pad2)
- removed copper zone on B.Cu, net Net-(R11-Pad1)
- removed copper zone on B.Cu, net Net-(R2-Pad2)
- removed copper zone on B.Cu, net Net-(R4-Pad2)
- removed copper zone on B.Cu, net Net-(R5-Pad2)
- removed copper zone on B.Cu, net Net-(R7-Pad2)
- removed copper zone on B.Cu, net TS+
- removed copper zone on F.Cu, net TS-
Other:
- board size 190.6 x 151.7 mm -> 123.5 x 151.7 mm
- board text removed: "0ADKC1000-BE ONLY please dont put some random fuse in"
- board text removed: "B+"
- board text removed: "B-"
- board text removed: "Charger +"
- board text removed: "Charger -"
- board text removed: "DCDC +"
- board text removed: "DCDC -"
- board text removed: "HIGH VOLTAGE"
- board text removed: "Please put kapton tape on the resistor base"
- board text removed: "Precharge Control Circuit Originally By Bill Yuan Updated by Gabriel Schoene"
- board text removed: "TO AIRS"
- board text removed: "TS+"
- board text removed: "TS_"
