File: Precharge Control Circuit/PCC/RTM.kicad_sch (KiCad schematic)
At the start: 34 parts, among them Q3 Q_NMOS_GSD, Q4 Q_NMOS_GSD, Q5 Q_NMOS_GSD, U10 4N35, U11 LM555xN, U9 TLV2372IP

Commit message: PCC finalized
Parts:
- removed DEBUG_1: LED, LED_THT:LED_D5.0mm, symbol Device:LED
- removed R64, R66, R68: 20k, Resistor_SMD:R_0805_2012Metric, symbol Device:R_US
- removed R74: 22k, Resistor_SMD:R_0805_2012Metric, symbol Device:R_US
- removed R76: 11k, Resistor_SMD:R_0805_2012Metric, symbol Device:R_US
- removed R77: 10k, Resistor_SMD:R_0805_2012Metric, symbol Device:R_US
- removed R_pullup1: 15k, Resistor_SMD:R_0805_2012Metric, symbol Device:R_US
- added R10, R11, R9: 10k, Resistor_SMD:R_0805_2012Metric, symbol Device:R_US
- added R15, R16: 20k, Resistor_SMD:R_0805_2012Metric, symbol Device:R_US
- added R4: 22k, Resistor_SMD:R_0805_2012Metric, symbol Device:R_US
- C27, C29, C30: MFG (none) -> KYOCERA AVX; MPN (none) -> 08055C104J4T4A
- C28: MFG (none) -> YAGEO; MPN (none) -> CC0805JKX7R9BB105
- DEBUG_2: MFG (none) -> Rohm Semiconductor; MPN (none) -> SLR-56VC3F
- R62: MFG (none) -> YAGEO; MPN (none) -> RC0805FR-0720KL
- R70: MFG (none) -> YAGEO; MPN (none) -> RC0805FR-7W10KL
- R73: MFG (none) -> Stackpole Electronics Inc; MPN (none) -> RPC0805JT22R0
- R75: MFG (none) -> YAGEO; MPN (none) -> RC0805FR-7W220KL
- U10: MFG (none) -> 4N35; MPN (none) -> Lite-On Inc.
- U12: value ~ -> (none)
Connections:
- net +12 ISO is gone; now on net 12V_UNISO: C31.2, C32.2, U12.6 (+Vout)
- net 12V_ISO: now also R4.1, R9.1
- net 12V_UNISO: now also R10.1, R11.1
- net Amber_LED: now also R9.2
- net V_BIAS: now also R10.2
- net V_SNS: now also R16.1
- net at Q3.1 (G), U9.1 (1OUT): now also R11.2
- net at R75.1, U11.7 (DIS): now also R4.2
- net at R62.1: now also R15.2
- new net: R15.1, R16.2
Other:
- note removed: "should be biased to 1.85 ohm"

Commit message: 2026 final
Other:
- note added: "NOTE THIS MUST NOW BE SWAPPED TO 5k from 10k"
Changed lines of the file:
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@@
+		)
+	)
+	(text "NOTE THIS MUST NOW BE SWAPPED TO 5k from 10k"
+		(exclude_from_sim no)
+		(at 135.255 45.085 0)
+		(effects
+			(font
+				(size 1.27 1.27)
+			)
 		)
 	)
