File: ESF Schematics/Charging TS_MZ_2026.kicad_sch (KiCad schematic)
At the start: 10 parts, among them SW2 B-AIR, SW4 B+ AIR

Commit message: 2026 final
Parts:
- removed R2, R3: 15k, symbol Device:R_US
- added F22, F39: (no value), symbol fuse:Fuse
- F21, F38: value ~ -> (none)
- F30: value ~ -> SPF J0100.X fuse
Connections:
- net at R4.1, SW2.2 (B): now also F22.; no longer F21.
- net at SW4.1 (A): now also F30.; no longer BT1.1 (+)
- net at F21.: now also F22.
- net at F38.: now also F39.
- net at R1.2: now also SW4.2 (B), F39.; no longer F30.
- new net: BT1.1 (+), F30.
Other:
- note added: "1.25A 0ADKC1250-BE"
- note added: "18 awg (0.82mm2) milspec wire"
- note added: "1A 0ADKC1000-BE"
- note added: "HV+"
- note added: "HV-"
- note added: "Rincon REC45B1Ja B+ IR"
- note added: "Rincon REC45B1Ja B- IR"
- note added: "SLPIPB50BS01EH HV in connector"
- note added: "fuse: 100A SPF J0100.X"
- note added: "no connector, gland wire passthrough Shielding terminates at gland"
- note removed: "18 awg (0.75mm2)"
- note removed: "AC-HA011042 & AC-HA015861 Accumulator HV out connector"
- note removed: "Green indicates contactor/terminal"
- note removed: "OADKC1000-BE 1A fuse inside MPD BF303 inline fuse holder"
- note removed: "Pack Fuse & MSD SPFJO9O.X fuse mounted inside a RL00571-250R"
- note removed: "Rincon_RXC159PA B+ AIR"
- note removed: "Rincon_RXC159PA B- AIR"
- note removed: "V+"
- note removed: "V-"
