File: ESF Schematics/Charging shutdown_MZ_2026.kicad_sch (KiCad schematic)
At the start: 15 parts, among them K2 Relay_DPST-NO, K3 Relay_DPST-NO

Commit message: 2026 final
Parts:
- removed JP5: Jumper_2_Open, symbol Jumper:Jumper_2_Open
Connections:
- net +12V: now also RST4.2
- net at JP4.2 (B): now also K3.23
Other:
- note added: "Battery Enclosure"
- note removed: "Accumulator Enclosure"
- note removed: "Charger-TS Interlock"
- note removed: "Safety Daisy Chain return since any interlock disconnect must stop charger"
