File: ESF Schematics/Shutdown_Circuit MZ 2026.kicad_sch (KiCad schematic)
At the start: 27 parts, among them K1 Relay_DPST-NO, K2 Relay_DPST-NO, K3 Relay_DPST-NO

Commit message: 2026 final
Parts:
- added 5A: Fuse, symbol Device:Fuse
- REC45B1Ja: renamed from RXC159PA; value AIR+ -> IR+
- REC45B1Ja: renamed from RXC159PA; value AIR- -> IR-
- renumbered 5A to 10A
Connections:
- net +12V: now also 5A.2; no longer 10A.2
- new net: 10A.2, 5A.1
Other:
- note removed: "(PCB fuse)"
