File: ESF Schematics/TS accu internal MZ 2026.kicad_sch (KiCad schematic)
At the start: 43 parts, among them SW1 B-AIR, SW2 B+ AIR, U1 RH3

Commit message: 2026 final
Parts:
- removed JP2: Jumper_2_Open, symbol Jumper:Jumper_2_Open
- removed R1, R3: 15k, symbol Device:R_US
- added F19, F29, F30, F31, F32, F33, F34, F35, F36: (no value), symbol fuse:Fuse
- added Pre-Resist2, Pre-Resist3: ## Ohm, symbol Device:R_US
- added SW3: SW_DPST_x2, symbol Switch:SW_DPST_x2
Connections:
- net at F7.: now also F3., F4., F6., F8., F9.
- net B-: now reaches F17.
- net at SW1.1 (A): now also F1., F2., F5.; no longer F17.
- net at F16.: now also SW3.1 (A)
- net at SW2.2 (B): no longer Pre-Resist1.1
- net B+: now reaches F18., U1.2
- net at SW2.1 (A): now also SW3.2 (B); no longer F18.
- net TS- unfused: now reaches E1. (HV-), U1.4
- net TS- unfused: now also F29., Pre-Resist2.2
- net at F22.: now also F20., F21., F23., F24., F25.
- new net: F19., F32., F33., F34., F35.
- new net: F16., F26., F27., F28.
- new net: F29., F30., F31., F36.
- new net: F10., F11., F12., F13., F14., F15.
- new net Energy Meter +: E1. (HV-), F34.
- new net HV indicator +: F32.
- new net HV indicator -: F31.
- new net IMD +: F33.
- new net IMD -: F30.
- new net RTM Light (internal): F35., F36.
- new net TS+ unfused: F19., Pre-Resist1.1, Pre-Resist3.2
- now unconnected: F10., F13., F25., F28., F5., F6.
Other:
- note added: "0.3mm 4.5oz traces"
- note added: "0679L3000-05 3A fuses"
- note added: "1.25A 0ADKC1250-BE inside 0031.8222 holder"
- note added: "100A SPFJ0100.X"
- note added: "10A fuse: 0505010.MXP inline housing: F10152-ND 20A rated OEM pigtail"
- note added: "10A fuse: 0505010.MXP inline housing: F10152-ND 20A rated pigtail"
- note added: "120mm unfused lenght (measured, pics provided on request)"
- note added: "127A"
- note added: "130mm wire measured pics provided on request"
- note added: "15k"
- note added: "16mm pcb trace"
- note added: "16mm trace"
- note added: "18 awg (0.82mm2) CF270-UL-07-04-D"
- note added: "18 awg (0.82mm2) milspec"
- note added: "19mm PCB trace"
- note added: "19mm to first fuse"
- note added: "19mm trace"
- note added: "2 series 2.7k RTO020F27000JTE3"
- note added: "242266 lugs"
- note added: "50mm2 wire 15-08565 Shielded at gland"
- note added: "5580850 lug for 50mm2 output"
- note added: "5mm trace to first fuse"
- note added: "94722-01-ND on IR ring terminal to milspec"
- note added: "94722-01-ND ring terminal"
- note added: "All internal wires are double wrapped in raychem"
- note added: "B- used for sense circuitry"
- note added: "Bussbar: 69.85mm2 6061 aluminum"
- note added: "Connector 1: 0462070206"
- note added: "Green indicates everything else (non 18awg wire, bussbar, PCB trace, or terminal)"
- note added: "High Voltage Board (HVB) All PCB traces are 2.5mm wide, 1oz copper"
- note added: "IPL1-106-01-L-S-RA-K connector OEM Orion wire"
- note added: "MSD EM30MSD"
- note added: "Maintinance plug 2043130010 female 2032630001 pin"
- note added: "Maintinance plug 2043130010 female 2032630001 pin 242266 lugs"
- note added: "RH3-12v Precharge/Discharge SPDT Discharge is NC Precharge is NO"
- note added: "Rincon REC45B1Ja B+ IR"
- note added: "Rincon REC45B1Ja B- IR"
- note added: "Voltage Indicator: PK-260-320-SJSJ"
- note added: "all above are 1A 0ADKC1000-BE inside 0031.8222 holder"
- note added: "all below are 1A 0ADKC1000-BE inside 0031.8222 holder"
- note added: "in this schematic All orange wires are high current path (35mm2/50mm2)"
- note added: "milspec"
- note added: "no external HV connectors shielding terminates at gland"
- note added: "output connector 2: 0039288120"
- note added: "ring terminal on EM: 94722-01-ND Wire: 18 awg milspec"
- note removed: "0679L2000-01 2A fuses"
- note removed: "140A"
- note removed: "?? Accumulator HV out connector"
- note removed: "CT4397-02-2 TSMP connector"
- note removed: "Green indicates everything else (other wire, bussbar, PCB trace, or terminal)"
- note removed: "IMD & RTM use 0ADKC1000-BE 1A fuse DCDC uses 0ADKC3150-BE 3.15A fuse inside MPD BF303 inline fuse holder"
- note removed: "MSD"
- note removed: "Molex Micro-fit(430452202) 22 pin connector 18 awg milspec wire"
- note removed: "RH3-12v Precharge/Discharge is SPDT Discharge is NC Precharge is NO"
- note removed: "RL00801-35 Maintinence plug"
- note removed: "Rincon RXC159PA B- AIR"
- note removed: "Rincon_RXC159PA B+ AIR"
- note removed: "Voltage indicator DH-670"
- note removed: "in this schematic All orange wires are 35mm2"
