File: ESF Schematics/TS external KZ 2025.kicad_sch (KiCad schematic)
At the start: 0 parts

Commit message: 2026 final
Other:
- note added: "All Inverter connections: SLPIPB50BSO1EH Sheilding terminates at inverter connector"
- note added: "All Inverter connections: SLPIPB50BSO1EH Sheilding terminates: connector on inverter"
- note added: "High Voltage Battery (HVB)"
- note added: "No connector, wire passes through gland to inside container"
- note added: "Sheild terminates at gland to HVB (No connector)"
- note added: "Sheilding terminates at gland to housing"
- note added: "Shield terminates at gland"
- note added: "TS+"
- note added: "TS-"
- note added: "TSMP Container"
- note added: "TSMP connector CT2910-2 Soldered Wire"
- note added: "TSMP wire: CF270-UL-07-04-D 18 awg (0.82mm2)"
- note added: "motor lug: 5580850 Shielding underminated"
- note removed: "AC-HA011042 & AC-HA015861 Accumulator HV out connector"
- note removed: "Accumulator"
- note removed: "Motor Connectors: LCMA50-6-L Lugs Out of Inverter: SurLok Plus EMI Plugs (non-keyed) SLPIPB50BSO1EH Straight"
- note removed: "Shield terminates in connector"
- note removed: "Shielding terminates at controller connectors"
- note removed: "SurLok Plus EMI Plugs SLPIPB50BSO1EH Straight Connector on HV+"
- note removed: "SurLok Plus EMI Plugs SLPIPB50BSO1EH Straight onnector on HV-"
- note removed: "TSMP connector CT2910-2"
- note removed: "motor controller shielding terminates at connector motor sheilding is terminated with copper braid to gnd"
Changed lines of the file:
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@@
 (kicad_sch
-	(version 20250114)
+	(version 20260306)
 	(generator "eeschema")
-	(generator_version "9.0")
+	(generator_version "10.0")
 	(paper "A4")
 	(arc
@@
 		)
 	)
+	(arc
+		(start 55.6489 91.4004)
+		(mid 57.6681 92.6969)
+		(end 59.6414 94.0622)
+		(stroke
+			(width 0)
+			(type default)
+		)
+		(fill
+			(type none)
+		)
+	)
 	(rectangle
 		(start 107.95 63.246)
@@
 		)
 	)
-	(arc
-		(start 101.6 93.98)
-		(mid 104.1097 92.6494)
-		(end 106.68 91.44)
-		(stroke
-			(width 0)
-			(type default)
-		)
-		(fill
-			(type none)
-		)
-	)
-	(text "Shielding terminates\nat controller connectors"
-		(exclude_from_sim no)
-		(at 95.25 72.39 0)
-		(effects
-			(font
-				(size 1.27 1.27)
-			)
-		)
-	)
-	(text "SurLok Plus EMI Plugs\nSLPIPB50BSO1EH Straight\nonnector\non HV-"
-		(exclude_from_sim no)
-		(at 93.218 99.314 0)
-		(effects
-			(font
-				(size 1.27 1.27)
-			)
-		)
-	)
-	(text "TSMP connector\nCT2910-2"
-		(exclude_from_sim no)
-		(at 42.672 57.15 0)
+	(rectangle
+		(start 35.306 39.878)
+		(end 50.546 49.022)
+		(stroke
+			(width 0)
+			(type dash_dot_dot)
+			(color 0 0 0 1)
+		)
+		(fill
+			(type color)
+			(color 255 255 194 1)
+		)
+	)
+	(text "TSMP Container"
+		(exclude_from_sim no)
+		(at 42.926 42.164 0)
+		(effects
+			(font
+				(size 1.27 1.27)
+			)
+		)
+	)
+	(text "Sheilding terminates \nat gland to housing"
+		(exclude_from_sim no)
+		(at 31.496 51.308 0)
+		(effects
+			(font
+				(size 1.27 1.27)
+			)
+		)
+	)
+	(text "All Inverter connections:\nSLPIPB50BSO1EH\nSheilding terminates:\nconnector on inverter"
+		(exclude_from_sim no)
+		(at 92.202 77.978 0)
+		(effects
+			(font
+				(size 1.27 1.27)
+			)
+		)
+	)
+	(text "No connector, wire passes \nthrough gland to inside container"
+		(exclude_from_sim no)
+		(at 72.136 93.98 0)
+		(effects
+			(font
+				(size 1.27 1.27)
+			)
+		)
+	)
+	(text "motor lug:\n5580850\nShielding underminated"
+		(exclude_from_sim no)
+		(at 155.448 92.71 0)
+		(effects
+			(font
+				(size 1.27 1.27)
+			)
+		)
+	)
+	(text "TSMP connector\nCT2910-2\nSoldered Wire"
+		(exclude_from_sim no)
+		(at 61.468 45.212 0)
 		(effects
 			(font
@@
 		)
 	)
+	(text "All Inverter connections:\nSLPIPB50BSO1EH\nSheilding terminates\nat inverter connector"
+		(exclude_from_sim no)
+		(at 137.668 72.136 0)
+		(effects
+			(font
+				(size 1.27 1.27)
+			)
+		)
+	)
+	(text "Sheild terminates \nat gland to HVB\n(No connector)"
+		(exclude_from_sim no)
+		(at 54.356 59.944 0)
+		(effects
+			(font
+				(size 1.27 1.27)
+			)
+		)
+	)
 	(text "HV-"
 		(exclude_from_sim no)
@@
 	(text "Motor Controller"
 		(exclude_from_sim no)
-		(at 116.84 74.93 0)
-		(effects
-			(font
-				(size 1.27 1.27)
-			)
-		)
-	)
-	(text "motor controller shielding \nterminates at connector\nmotor sheilding is terminated \nwith copper braid to gnd"
-		(exclude_from_sim no)
-		(at 140.97 92.71 0)
-		(effects
-			(font
-				(size 1.27 1.27)
-			)
-		)
-	)
-	(text "HV-"
+		(at 116.078 74.676 0)
+		(effects
+			(font
+				(size 1.27 1.27)
+			)
+		)
+	)
+	(text "TSMP wire:\nCF270-UL-07-04-D\n18 awg (0.82mm2)"
+		(exclude_from_sim no)
+		(at 30.226 59.182 0)
+		(effects
+			(font
+				(size 1.27 1.27)
+			)
+		)
+	)
+	(text "TS-"
 		(exclude_from_sim no)
 		(at 46.99 92.71 0)
@@
 		)
 	)
-	(text "HV+"
+	(text "TS+"
 		(exclude_from_sim no)
 		(at 46.99 86.36 0)
@@
 		)
 	)
-	(text "Accumulator"
-		(exclude_from_sim no)
-		(at 30.48 83.82 0)
-		(effects
-			(font
-				(size 1.27 1.27)
-			)
-		)
-	)
-	(text "SurLok Plus EMI Plugs\nSLPIPB50BSO1EH Straight\nConnector\non HV+"
-		(exclude_from_sim no)
-		(at 93.726 80.772 0)
+	(text "High Voltage Battery (HVB)"
+		(exclude_from_sim no)
+		(at 32.258 83.566 0)
 		(effects
 			(font
@@
 		)
 	)
-	(text "AC-HA011042 & AC-HA015861\nAccumulator HV out connector"
-		(exclude_from_sim no)
-		(at 67.31 93.98 0)
-		(effects
-			(font
-				(size 1.016 1.016)
-			)
-		)
-	)
 	(text "TSMP Resistors \ninside accumulator"
 		(exclude_from_sim no)
@@
 		)
 	)
-	(text "Motor Connectors:\nLCMA50-6-L Lugs\n\nOut of Inverter:\nSurLok Plus EMI Plugs (non-keyed)\nSLPIPB50BSO1EH Straight"
-		(exclude_from_sim no)
-		(at 128.524 70.612 0)
-		(effects
-			(font
-				(size 1.016 1.016)
-			)
-			(justify left)
-		)
-	)
 	(text "50mm2\n"
 		(exclude_from_sim no)
@@
 		)
 	)
-	(text "Shield terminates \nin connector"
-		(exclude_from_sim no)
-		(at 64.77 80.01 0)
+	(text "Shield terminates \nat gland"
+		(exclude_from_sim no)
+		(at 64.77 84.074 0)
 		(effects
 			(font
@@
 	(wire
 		(pts
-			(xy 41.91 60.96) (xy 41.91 64.77)
+			(xy 44.196 47.498) (xy 44.196 63.5)
 		)
 		(stroke
@@
 	(wire
 		(pts
+			(xy 41.656 44.704) (xy 41.656 63.5)
+		)
+		(stroke
+			(width 0)
+			(type default)
+			(color 255 155 0 1)
+		)
+	)
+	(wire
+		(pts
+			(xy 41.656 44.704) (xy 52.324 44.704)
+		)
+		(stroke
+			(width 0)
+			(type default)
+			(color 255 155 0 1)
+		)
+	)
+	(wire
+		(pts
 			(xy 49.53 87.63) (xy 55.88 87.63)
 		)
@@
 	(wire
 		(pts
-			(xy 44.45 64.77) (xy 44.45 60.96)
-		)
-		(stroke
+			(xy 44.196 47.498) (xy 52.324 47.498)
+		)
+		(stroke
